File: hardware/power-board/PB-100/kicad/sheets/can1-safety.kicad_sch (KiCad schematic)
At the start: 0 parts

Commit message: Capture preliminary PB-100 schematic sheets
Parts:
- added JP_CAN1, U_CAN1: CAN1_TX_DISABLE_PRELIM, symbol PB100:PB100_CAN1_TX_DISABLE_PRELIM
Connections:
- new net CAN1_RX_ROUTE: JP_CAN1.4 (CAN1_RX_ROUTE), U_CAN1.4 (CAN1_RX_ROUTE)
- new net CAN1_TX_DISABLED_STATUS: JP_CAN1.2 (CAN1_TX_DISABLED_STATUS), U_CAN1.2 (CAN1_TX_DISABLED_STATUS)
- new net CAN1_TX_DISABLE_CMD: JP_CAN1.1 (CAN1_TX_DISABLE_CMD), U_CAN1.1 (CAN1_TX_DISABLE_CMD)
- new net CAN1_TX_ROUTE: JP_CAN1.3 (CAN1_TX_ROUTE), U_CAN1.3 (CAN1_TX_ROUTE)
- new net GND: JP_CAN1.5 (GND), U_CAN1.5 (GND)
Other:
- note added: "CAN1 safety capture notes: - Source traces: PB-100-can1-tx-disable-trace.csv, PB-100-can1-tx-disable.md, PB-100-can1-safety-verification.csv, PB-100-can1-production-dnp-review.csv, PB-100-schematic-net-domain-plan.csv - CAN1_TX_ROUTE remains DNP/open by default with no default-populated TX - CAN1_TX_DISABLED_STATUS remains visible to LB-100 as physical disabled state readback - Future vehicle-CAN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"
- note removed: "CAN1 safety capture notes: - Source trace: PB-100-can1-tx-disable-trace.csv - Production DNP review: PB-100-can1-production-dnp-review.csv - JP_CAN1 is the DNP/open physical missing-link in CAN1_TX_ROUTE - U_CAN1 is the optional default-disabled gate or silent-control element - CAN1_TX_ROUTE has no default-populated TX item - CAN1_TX_DISABLE_CMD defaults to disable by hardware pull - CAN1_TX_DISA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"
Changed lines of the file:
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@@
   (title_block
     (title "PB-100 CAN1 Safety")
-    (date "2026-06-30")
-    (rev "sheet-placeholder")
+    (date "2026-07-16")
+    (rev "preliminary-capture")
     (company "SVC Platform")
-    (comment 9 "Work queue: CAP-CAN1. CAN1 capture keeps TX DNP/open and future ADR only.")
-    (comment 1 "Capture contract: JP_CAN1 DNP/open TX link and U_CAN1 default-disabled gate.")
-    (comment 2 "Sources: PB-100-can1-tx-disable-trace.csv, PB-100-can1-production-dnp-review.csv, and PB-100-can1-tx-disable.md.")
+    (comment 9 "Work queue: CAP-CAN1. Preliminary schematic capture follows PB-100-schematic-capture-work-queue.csv.")
+    (comment 1 "Preliminary capture for CAN1 TX-disable readback and DNP/open TX path.")
+    (comment 2 "Sources: PB-100-can1-tx-disable-trace.csv, PB-100-can1-tx-disable.md, PB-100-can1-safety-verification.csv, PB-100-can1-production-dnp-review.csv.")
   )
-  (text "CAN1 safety capture notes:\n- Source trace: PB-100-can1-tx-disable-trace.csv\n- Production DNP review: PB-100-can1-production-dnp-review.csv\n- JP_CAN1 is the DNP/open physical missing-link in CAN1_TX_ROUTE\n- U_CAN1 is the optional default-disabled gate or silent-control element\n- CAN1_TX_ROUTE has no default-populated TX item\n- CAN1_TX_DISABLE_CMD defaults to disable by hardware pull\n- CAN1_TX_DISABLED_STATUS reflects physical disabled state and is visible to LB-100\n- CAN1_RX_ROUTE may be populated independently if CAN1 crosses PB-100\n- Any CAN1 TX enable path requires a future ADR and hardware action\n\nRev.1 firmware must not transmit on vehicle CAN."
-    (at 25 30 0)
+  (text "CAN1 safety capture notes:\n- Source traces: PB-100-can1-tx-disable-trace.csv, PB-100-can1-tx-disable.md, PB-100-can1-safety-verification.csv, PB-100-can1-production-dnp-review.csv, PB-100-schematic-net-domain-plan.csv\n- CAN1_TX_ROUTE remains DNP/open by default with no default-populated TX\n- CAN1_TX_DISABLED_STATUS remains visible to LB-100 as physical disabled state readback\n- Future vehicle-CAN TX requires a new ADR and explicit hardware action\n\nNo PCB layout from this preliminary capture."
+    (at 20 20 0)
     (effects (font (size 2.0 2.0)) (justify left top))
   )
+  (symbol
+    (lib_id "PB100:PB100_CAN1_TX_DISABLE_PRELIM")
+    (at 76.20 60.96 0)
+    (unit 1)
+    (exclude_from_sim no)
+    (in_bom yes)
+    (on_board yes)
+    (dnp yes)
+    (property "Reference" "JP_CAN1" (at 76.20 53.34 0) (effects (font (size 1.27 1.27))))
+    (property "Value" "CAN1_TX_DISABLE_PRELIM" (at 76.20 55.88 0) (effects (font (size 1.27 1.27))))
+    (property "Footprint" "" (at 76.20 68.58 0) (effects (font (size 1.27 1.27)) hide))
+    (property "Datasheet" "../PB-100-schematic-capture-plan.md" (at 76.20 71.12 0) (effects (font (size 1.27 1.27)) hide))
+    (pin "1")
+    (pin "2")
+    (pin "3")
+    (pin "4")
+    (pin "5")
+    (instances
+      (project "PB-100"
+        (path "/1af68b81-10b0-5461-9124-39421a2a6932/5cace8c6-5dc9-50ce-8c5f-35b8341c23b7/"
+          (reference "JP_CAN1")
+          (unit 1)
+        )
+      )
+    )
+  )
+  (wire (pts (xy 55.88 55.88) (xy 48.26 55.88)) (stroke (width 0) (type default)))
+  (global_label "CAN1_TX_DISABLE_CMD" (shape bidirectional) (at 48.26 55.88 0) (fields_autoplaced) (effects (font (size 1.27 1.27)) (justify right)) (property "Intersheetrefs" "${INTERSHEET_REFS}" (at 48.26 55.88 0) (effects (font (size 1.27 1.27)) hide)))
+  (wire (pts (xy 96.52 55.88) (xy 104.14 55.88)) (stroke (width 0) (type default)))
+  (global_label "CAN1_TX_DISABLED_STATUS" (shape bidirectional) (at 104.14 55.88 0) (fields_autoplaced) (effects (font (size 1.27 1.27)) (justify left)) (property "Intersheetrefs" "${INTERSHEET_REFS}" (at 104.14 55.88 0) (effects (font (size 1.27 1.27)) hide)))
+  (wire (pts (xy 55.88 60.96) (xy 48.26 60.96)) (stroke (width 0) (type default)))
+  (global_label "CAN1_TX_ROUTE" (shape bidirectional) (at 48.26 60.96 0) (fields_autoplaced) (effects (font (size 1.27 1.27)) (justify right)) (property "Intersheetrefs" "${INTERSHEET_REFS}" (at 48.26 60.96 0) (effects (font (size 1.27 1.27)) hide)))
+  (wire (pts (xy 96.52 60.96) (xy 104.14 60.96)) (stroke (width 0) (type default)))
+  (global_label "CAN1_RX_ROUTE" (shape bidirectional) (at 104.14 60.96 0) (fields_autoplaced) (effects (font (size 1.27 1.27)) (justify left)) (property "Intersheetrefs" "${INTERSHEET_REFS}" (at 104.14 60.96 0) (effects (font (size 1.27 1.27)) hide)))
+  (wire (pts (xy 55.88 66.04) (xy 48.26 66.04)) (stroke (width 0) (type default)))
+  (global_label "GND" (shape bidirectional) (at 48.26 66.04 0) (fields_autoplaced) (effects (font (size 1.27 1.27)) (justify right)) (property "Intersheetrefs" "${INTERSHEET_REFS}" (at 48.26 66.04 0) (effects (font (size 1.27 1.27)) hide)))
+  (symbol
+    (lib_id "PB100:PB100_CAN1_TX_DISABLE_PRELIM")
+    (at 152.40 60.96 0)
+    (unit 1)
+    (exclude_from_sim no)
+    (in_bom yes)
+    (on_board yes)
+    (dnp no)
+    (property "Reference" "U_CAN1" (at 152.40 53.34 0) (effects (font (size 1.27 1.27))))
+    (property "Value" "CAN1_TX_DISABLE_PRELIM" (at 152.40 55.88 0) (effects (font (size 1.27 1.27))))
+    (property "Footprint" "" (at 152.40 68.58 0) (effects (font (size 1.27 1.27)) hide))
+    (property "Datasheet" "../PB-100-schematic-capture-plan.md" (at 152.40 71.12 0) (effects (font (size 1.27 1.27)) hide))
+    (pin "1")
+    (pin "2")
+    (pin "3")
+    (pin "4")
+    (pin "5")
+    (instances
+      (project "PB-100"
+        (path "/1af68b81-10b0-5461-9124-39421a2a6932/a9a77c70-6457-523b-8ead-86fe8f88fa3e/"
+          (reference "U_CAN1")
+          (unit 1)
+        )
+      )
+    )
+  )
+  (wire (pts (xy 132.08 55.88) (xy 124.46 55.88)) (stroke (width 0) (type default)))
+  (global_label "CAN1_TX_DISABLE_CMD" (shape bidirectional) (at 124.46 55.88 0) (fields_autoplaced) (effects (font (size 1.27 1.27)) (justify right)) (property "Intersheetrefs" "${INTERSHEET_REFS}" (at 124.46 55.88 0) (effects (font (size 1.27 1.27)) hide)))
+  (wire (pts (xy 172.72 55.88) (xy 180.34 55.88)) (stroke (width 0) (type default)))
+  (global_label "CAN1_TX_DISABLED_STATUS" (shape bidirectional) (at 180.34 55.88 0) (fields_autoplaced) (effects (font (size 1.27 1.27)) (justify left)) (property "Intersheetrefs" "${INTERSHEET_REFS}" (at 180.34 55.88 0) (effects (font (size 1.27 1.27)) hide)))
+  (wire (pts (xy 132.08 60.96) (xy 124.46 60.96)) (stroke (width 0) (type default)))
+  (global_label "CAN1_TX_ROUTE" (shape bidirectional) (at 124.46 60.96 0) (fields_autoplaced) (effects (font (size 1.27 1.27)) (justify right)) (property "Intersheetrefs" "${INTERSHEET_REFS}" (at 124.46 60.96 0) (effects (font (size 1.27 1.27)) hide)))
+  (wire (pts (xy 172.72 60.96) (xy 180.34 60.96)) (stroke (width 0) (type default)))
+  (global_label "CAN1_RX_ROUTE" (shape bidirectional) (at 180.34 60.96 0) (fields_autoplaced) (effects (font (size 1.27 1.27)) (justify left)) (property "Intersheetrefs" "${INTERSHEET_REFS}" (at 180.34 60.96 0) (effects (font (size 1.27 1.27)) hide)))
+  (wire (pts (xy 132.08 66.04) (xy 124.46 66.04)) (stroke (width 0) (type default)))
+  (global_label "GND" (shape bidirectional) (at 124.46 66.04 0) (fields_autoplaced) (effects (font (size 1.27 1.27)) (justify right)) (property "Intersheetrefs" "${INTERSHEET_REFS}" (at 124.46 66.04 0) (effects (font (size 1.27 1.27)) hide)))
+  (symbol
+    (lib_id "PB100:PB100_ERC_SIGNAL_DRIVER_PRELIM")
+    (at 15.24 20.32 0)
+    (unit 1)
+    (exclude_from_sim no)
+    (in_bom no)
+    (on_board no)
+    (dnp no)
+    (property "Reference" "#DRV001" (at 15.24 17.78 0) (effects (font (size 1.27 1.27))))
+    (property "Value" "PB100_ERC_SIGNAL_DRIVER_PRELIM" (at 15.24 22.86 0) (effects (font (size 1.27 1.27))))
+    (property "Footprint" "" (at 15.24 25.40 0) (effects (font (size 1.27 1.27)) hide))
+    (property "Datasheet" "../PB-100-schematic-capture-plan.md" (at 15.24 27.94 0) (effects (font (size 1.27 1.27)) hide))
+    (pin "1")
+  )
+  (global_label "CAN1_TX_DISABLE_CMD" (shape bidirectional) (at 15.24 20.32 0) (fields_autoplaced) (effects (font (size 1.27 1.27)) (justify left)) (property "Intersheetrefs" "${INTERSHEET_REFS}" (at 15.24 20.32 0) (effects (font (size 1.27 1.27)) hide)))
+  (symbol
+    (lib_id "PB100:PB100_ERC_SIGNAL_DRIVER_PRELIM")
+    (at 15.24 25.40 0)
+    (unit 1)
+    (exclude_from_sim no)
+    (in_bom no)
+    (on_board no)
+    (dnp no)
+    (property "Reference" "#DRV002" (at 15.24 22.86 0) (effects (font (size 1.27 1.27))))
+    (property "Value" "PB100_ERC_SIGNAL_DRIVER_PRELIM" (at 15.24 27.94 0) (effects (font (size 1.27 1.27))))
+    (property "Footprint" "" (at 15.24 30.48 0) (effects (font (size 1.27 1.27)) hide))
+    (property "Datasheet" "../PB-100-schematic-capture-plan.md" (at 15.24 33.02 0) (effects (font (size 1.27 1.27)) hide))
+    (pin "1")
+  )
+  (global_label "CAN1_TX_ROUTE" (shape bidirectional) (at 15.24 25.40 0) (fields_autoplaced) (effects (font (size 1.27 1.27)) (justify left)) (property "Intersheetrefs" "${INTERSHEET_REFS}" (at 15.24 25.40 0) (effects (font (size 1.27 1.27)) hide)))
+  (symbol
+    (lib_id "PB100:PB100_ERC_POWER_FLAG_PRELIM")
+    (at 15.24 30.48 0)
+    (unit 1)
+    (exclude_from_sim no)
+    (in_bom no)
+    (on_board no)
+    (dnp no)
+    (property "Reference" "#PWR003" (at 15.24 27.94 0) (effects (font (size 1.27 1.27))))
+    (property "Value" "PB100_ERC_POWER_FLAG_PRELIM" (at 15.24 33.02 0) (effects (font (size 1.27 1.27))))
+    (property "Footprint" "" (at 15.24 35.56 0) (effects (font (size 1.27 1.27)) hide))
+    (property "Datasheet" "../PB-100-schematic-capture-plan.md" (at 15.24 38.10 0) (effects (font (size 1.27 1.27)) hide))
+    (pin "1")
+  )
+  (global_label "GND" (shape bidirectional) (at 15.24 30.48 0) (fields_autoplaced) (effects (font (size 1.27 1.27)) (justify left)) (property "Intersheetrefs" "${INTERSHEET_REFS}" (at 15.24 30.48 0) (effects (font (size 1.27 1.27)) hide)))
 )

Commit message: Add PB-100 CAN1 reset bench checklist
Other:
- note added: "CAN1 safety capture notes: - Source traces: PB-100-can1-tx-disable-trace.csv, PB-100-can1-tx-disable.md, PB-100-can1-safety-verification.csv, PB-100-can1-production-dnp-review.csv, PB-100-can1-reset-bench-checklist.csv, PB-100-schematic-net-domain-plan.csv - CAN1_TX_ROUTE remains DNP/open by default with no default-populated TX - CAN1_TX_DISABLED_STATUS remains visible to LB-100 as physical disab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"
- note removed: "CAN1 safety capture notes: - Source traces: PB-100-can1-tx-disable-trace.csv, PB-100-can1-tx-disable.md, PB-100-can1-safety-verification.csv, PB-100-can1-production-dnp-review.csv, PB-100-schematic-net-domain-plan.csv - CAN1_TX_ROUTE remains DNP/open by default with no default-populated TX - CAN1_TX_DISABLED_STATUS remains visible to LB-100 as physical disabled state readback - Future vehicle-CAN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"
Changed lines of the file:
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@@
     (comment 2 "Sources: PB-100-can1-tx-disable-trace.csv, PB-100-can1-tx-disable.md, PB-100-can1-safety-verification.csv, PB-100-can1-production-dnp-review.csv.")
   )
-  (text "CAN1 safety capture notes:\n- Source traces: PB-100-can1-tx-disable-trace.csv, PB-100-can1-tx-disable.md, PB-100-can1-safety-verification.csv, PB-100-can1-production-dnp-review.csv, PB-100-schematic-net-domain-plan.csv\n- CAN1_TX_ROUTE remains DNP/open by default with no default-populated TX\n- CAN1_TX_DISABLED_STATUS remains visible to LB-100 as physical disabled state readback\n- Future vehicle-CAN TX requires a new ADR and explicit hardware action\n\nNo PCB layout from this preliminary capture."
+  (text "CAN1 safety capture notes:\n- Source traces: PB-100-can1-tx-disable-trace.csv, PB-100-can1-tx-disable.md, PB-100-can1-safety-verification.csv, PB-100-can1-production-dnp-review.csv, PB-100-can1-reset-bench-checklist.csv, PB-100-schematic-net-domain-plan.csv\n- CAN1_TX_ROUTE remains DNP/open by default with no default-populated TX\n- CAN1_TX_DISABLED_STATUS remains visible to LB-100 as physical disabled state readback\n- PB-BENCH-012 covers reset, unpowered, DNP/open, and disabled-status checks\n- Future vehicle-CAN TX requires a new ADR and explicit hardware action\n\nNo PCB layout from this preliminary capture."
     (at 20 20 0)
     (effects (font (size 2.0 2.0)) (justify left top))

Commit message: Add PB-100 CAN1 default-disable freeze checklist
Other:
- note added: "CAN1 safety capture notes: - Source traces: PB-100-can1-tx-disable-trace.csv, PB-100-can1-tx-disable.md, PB-100-can1-safety-verification.csv, PB-100-can1-production-dnp-review.csv, PB-100-can1-default-disable-freeze-checklist.csv, PB-100-can1-reset-bench-checklist.csv, PB-100-schematic-net-domain-plan.csv - CAN1_TX_ROUTE remains DNP/open by default with no default-populated TX - CAN1_TX_DISABLED_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"
- note removed: "CAN1 safety capture notes: - Source traces: PB-100-can1-tx-disable-trace.csv, PB-100-can1-tx-disable.md, PB-100-can1-safety-verification.csv, PB-100-can1-production-dnp-review.csv, PB-100-can1-reset-bench-checklist.csv, PB-100-schematic-net-domain-plan.csv - CAN1_TX_ROUTE remains DNP/open by default with no default-populated TX - CAN1_TX_DISABLED_STATUS remains visible to LB-100 as physical disab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"
Changed lines of the file:
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@@
     (comment 9 "Work queue: CAP-CAN1. Preliminary schematic capture follows PB-100-schematic-capture-work-queue.csv.")
     (comment 1 "Preliminary capture for CAN1 TX-disable readback and DNP/open TX path.")
-    (comment 2 "Sources: PB-100-can1-tx-disable-trace.csv, PB-100-can1-tx-disable.md, PB-100-can1-safety-verification.csv, PB-100-can1-production-dnp-review.csv.")
+    (comment 2 "Sources: PB-100-can1-tx-disable-trace.csv, PB-100-can1-tx-disable.md, PB-100-can1-safety-verification.csv, PB-100-can1-production-dnp-review.csv, PB-100-can1-default-disable-freeze-checklist.csv.")
   )
-  (text "CAN1 safety capture notes:\n- Source traces: PB-100-can1-tx-disable-trace.csv, PB-100-can1-tx-disable.md, PB-100-can1-safety-verification.csv, PB-100-can1-production-dnp-review.csv, PB-100-can1-reset-bench-checklist.csv, PB-100-schematic-net-domain-plan.csv\n- CAN1_TX_ROUTE remains DNP/open by default with no default-populated TX\n- CAN1_TX_DISABLED_STATUS remains visible to LB-100 as physical disabled state readback\n- PB-BENCH-012 covers reset, unpowered, DNP/open, and disabled-status checks\n- Future vehicle-CAN TX requires a new ADR and explicit hardware action\n\nNo PCB layout from this preliminary capture."
+  (text "CAN1 safety capture notes:\n- Source traces: PB-100-can1-tx-disable-trace.csv, PB-100-can1-tx-disable.md, PB-100-can1-safety-verification.csv, PB-100-can1-production-dnp-review.csv, PB-100-can1-default-disable-freeze-checklist.csv, PB-100-can1-reset-bench-checklist.csv, PB-100-schematic-net-domain-plan.csv\n- CAN1_TX_ROUTE remains DNP/open by default with no default-populated TX\n- CAN1_TX_DISABLED_STATUS remains visible to LB-100 as physical disabled state readback\n- PB-BENCH-012 covers reset, unpowered, DNP/open, and disabled-status checks\n- Future vehicle-CAN TX requires a new ADR and explicit hardware action\n\nNo PCB layout from this preliminary capture."
     (at 20 20 0)
     (effects (font (size 2.0 2.0)) (justify left top))
