File: hardware/power-board/PB-100/kicad/sheets/b2b-interface.kicad_sch (KiCad schematic)
At the start: 1 part

Commit message: Add PB-100 B2B interface freeze checklist
Other:
- note added: "B2B interface capture notes: - Source traces: PB-100-b2b-interface-trace.csv, PB-100-b2b-lb100-resource-binding.csv, PB-100-b2b-lb100-pin-audit-checklist.csv, PB-100-b2b-interface-freeze-checklist.csv, PB-100-b2b-pin-map.csv, PB-100-b2b-pin-budget.csv - JPB1 candidates FX18-100P-0.8SV10 and FX18-100S-0.8SV20 carry power, output controls, faults, current telemetry, board telemetry, CAN1 safety, an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"
- note removed: "B2B interface capture notes: - Source traces: PB-100-b2b-interface-trace.csv, PB-100-b2b-lb100-resource-binding.csv, PB-100-b2b-lb100-pin-audit-checklist.csv, PB-100-b2b-pin-map.csv, PB-100-b2b-pin-budget.csv - JPB1 candidates FX18-100P-0.8SV10 and FX18-100S-0.8SV20 carry power, output controls, faults, current telemetry, board telemetry, CAN1 safety, and reserves - Exact LB-100 MCU pin binding a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"
Changed lines of the file:
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@@
     (comment 9 "Work queue: CAP-B2B. Preliminary schematic capture follows PB-100-schematic-capture-work-queue.csv.")
     (comment 1 "Preliminary capture for JPB1 100-pin FX18 candidate interface.")
-    (comment 2 "Sources: PB-100-b2b-interface-trace.csv, PB-100-b2b-lb100-resource-binding.csv, PB-100-b2b-lb100-pin-audit-checklist.csv, and PB-100-b2b-pin-map.csv.")
+    (comment 2 "Sources: PB-100-b2b-interface-trace.csv, PB-100-b2b-lb100-resource-binding.csv, PB-100-b2b-lb100-pin-audit-checklist.csv, PB-100-b2b-interface-freeze-checklist.csv, and PB-100-b2b-pin-map.csv.")
   )
-  (text "B2B interface capture notes:\n- Source traces: PB-100-b2b-interface-trace.csv, PB-100-b2b-lb100-resource-binding.csv, PB-100-b2b-lb100-pin-audit-checklist.csv, PB-100-b2b-pin-map.csv, PB-100-b2b-pin-budget.csv\n- JPB1 candidates FX18-100P-0.8SV10 and FX18-100S-0.8SV20 carry power, output controls, faults, current telemetry, board telemetry, CAN1 safety, and reserves\n- Exact LB-100 MCU pin binding and FX18 footprint drawing audit remain schematic-freeze work\n\nNo PCB layout from this preliminary capture."
+  (text "B2B interface capture notes:\n- Source traces: PB-100-b2b-interface-trace.csv, PB-100-b2b-lb100-resource-binding.csv, PB-100-b2b-lb100-pin-audit-checklist.csv, PB-100-b2b-interface-freeze-checklist.csv, PB-100-b2b-pin-map.csv, PB-100-b2b-pin-budget.csv\n- JPB1 candidates FX18-100P-0.8SV10 and FX18-100S-0.8SV20 carry power, output controls, faults, current telemetry, board telemetry, CAN1 safety, and reserves\n- Exact LB-100 MCU pin binding and FX18 footprint drawing audit remain schematic-freeze work\n\nNo PCB layout from this preliminary capture."
     (at 20 20 0)
     (effects (font (size 2.0 2.0)) (justify left top))
