File: hardware/power-board/PB-100/kicad/sheets/input-protection.kicad_sch (KiCad schematic)
At the start: 6 parts, among them J1 INPUT_CONNECTOR_CLASS_PRELIM, Q1 INPUT_NMOS_TOLL_PRELIM, U1 LM74700QDBVRQ1_PRELIM, U2 INA228_Q1_PRELIM

Commit message: Add PB-100 input reverse Q1 derivation precheck
Other:
- note added: "Input protection capture notes: - Source traces: PB-100-input-reverse-package-trace.csv, PB-100-input-reverse-freeze-review.csv, PB-100-input-reverse-q1-freeze-checklist.csv, PB-100-input-reverse-q1-derivation-precheck.csv, PB-100-board-current-budget-trace.csv, PB-100-board-current-budget-freeze-review.csv, PB-100-board-current-budget-design-calculation.md, PB-100-board-current-budget-value-free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"
- note removed: "Input protection capture notes: - Source traces: PB-100-input-reverse-package-trace.csv, PB-100-input-reverse-freeze-review.csv, PB-100-input-reverse-q1-freeze-checklist.csv, PB-100-board-current-budget-trace.csv, PB-100-board-current-budget-freeze-review.csv, PB-100-board-current-budget-design-calculation.md, PB-100-board-current-budget-value-freeze-checklist.csv, PB-100-tvs-load-dump-margin-tra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"
Changed lines of the file:
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@@
     (comment 9 "Work queue: CAP-INP. Preliminary schematic capture follows PB-100-schematic-capture-work-queue.csv.")
     (comment 1 "Preliminary capture for battery input, TVS, reverse protection, input telemetry.")
-    (comment 2 "Sources: PB-100-input-reverse-package-trace.csv, PB-100-input-reverse-freeze-review.csv, PB-100-input-reverse-q1-freeze-checklist.csv, PB-100-board-current-budget-trace.csv, PB-100-board-current-budget-freeze-review.csv, PB-100-board-current-budget-design-calculation.md, PB-100-board-current-budget-value-freeze-checklist.csv, PB-100-tvs-load-dump-margin-trace.csv, PB-100-tvs-load-dump-freeze-review.csv, PB-100-tvs-overshoot-escape-checklist.csv.")
+    (comment 2 "Sources: PB-100-input-reverse-package-trace.csv, PB-100-input-reverse-freeze-review.csv, PB-100-input-reverse-q1-freeze-checklist.csv, PB-100-input-reverse-q1-derivation-precheck.csv, PB-100-board-current-budget-trace.csv, PB-100-board-current-budget-freeze-review.csv, PB-100-board-current-budget-design-calculation.md, PB-100-board-current-budget-value-freeze-checklist.csv, PB-100-tvs-load-dump-margin-trace.csv, PB-100-tvs-load-dump-freeze-review.csv, PB-100-tvs-overshoot-escape-checklist.csv.")
   )
-  (text "Input protection capture notes:\n- Source traces: PB-100-input-reverse-package-trace.csv, PB-100-input-reverse-freeze-review.csv, PB-100-input-reverse-q1-freeze-checklist.csv, PB-100-board-current-budget-trace.csv, PB-100-board-current-budget-freeze-review.csv, PB-100-board-current-budget-design-calculation.md, PB-100-board-current-budget-value-freeze-checklist.csv, PB-100-tvs-load-dump-margin-trace.csv, PB-100-tvs-load-dump-freeze-review.csv, PB-100-tvs-overshoot-escape-checklist.csv\n- VBAT_RAW before reverse protection\n- VBAT_PROT after reverse protection\n- D1 input TVS candidate\n- U1 LM74700-class controller\n- Q1 dedicated input MOSFET strategy\n- RSH1/U2 total input current monitor\n- 40 A review covers connector derating, shunt Kelvin path, Q1 thermal path, firmware config, and no-layout boundary\n\nNo PCB layout from this preliminary capture."
+  (text "Input protection capture notes:\n- Source traces: PB-100-input-reverse-package-trace.csv, PB-100-input-reverse-freeze-review.csv, PB-100-input-reverse-q1-freeze-checklist.csv, PB-100-input-reverse-q1-derivation-precheck.csv, PB-100-board-current-budget-trace.csv, PB-100-board-current-budget-freeze-review.csv, PB-100-board-current-budget-design-calculation.md, PB-100-board-current-budget-value-freeze-checklist.csv, PB-100-tvs-load-dump-margin-trace.csv, PB-100-tvs-load-dump-freeze-review.csv, PB-100-tvs-overshoot-escape-checklist.csv\n- VBAT_RAW before reverse protection\n- VBAT_PROT after reverse protection\n- D1 input TVS candidate\n- U1 LM74700-class controller\n- Q1 dedicated input MOSFET strategy\n- RSH1/U2 total input current monitor\n- 40 A review covers connector derating, shunt Kelvin path, Q1 thermal path, firmware config, and no-layout boundary\n\nNo PCB layout from this preliminary capture."
     (at 20 20 0)
     (effects (font (size 2.0 2.0)) (justify left top))
