File: hardware/power-board/PB-100/kicad/sheets/input-protection.kicad_sch (KiCad schematic)
At the start: 14 parts, among them J1 INPUT_CONNECTOR_CLASS_PRELIM, Q1 IAUT300N08S5N012ATMA2, Q2 IAUTN15S6N025ATMA1, U1 LM74930QRGERQ1, U2 INA228_Q1_PRELIM

Commit message: Advance PB-100 EVT routing baseline
Parts:
- removed CCAP1: 100nF 25V X7R, symbol PB100:PB100_TWO_PIN_COMPONENT
- removed CVS1: CGA6N3X7R2A225M230AE 2.2uF 100V X7R; Ceff>=1uF@56V, symbol PB100:PB100_TWO_PIN_COMPONENT
- removed D1: SM8S33AHM3/I, PB100:DO-218AC_Vishay_SM8S, symbol PB100:PB100_SM8S33AHM3I
- removed DZVS1: 56V automotive Zener, symbol PB100:PB100_TWO_PIN_COMPONENT
- removed J1: INPUT_CONNECTOR_CLASS_PRELIM, symbol PB100:PB100_INPUT_CONNECTOR_CLASS_PRELIM
- removed Q1: IAUT300N08S5N012ATMA2, PB100:PG-HSOF-8-1_TOLL_Infineon, symbol PB100:PB100_POWER_NMOS_TOLL_80V
- removed Q2: IAUTN15S6N025ATMA1, PB100:PG-HSOF-8-1_TOLL_Infineon, symbol PB100:PB100_POWER_NMOS_TOLL_150V
- removed R3, R4: 42.2k 1%, symbol PB100:PB100_TWO_PIN_COMPONENT
- removed R5: 1.00k 1%, symbol PB100:PB100_TWO_PIN_COMPONENT
- removed R6: 10k 1%, symbol PB100:PB100_TWO_PIN_COMPONENT
- removed RSH1: INPUT_SHUNT_PRELIM, symbol PB100:PB100_INPUT_SHUNT_PRELIM
- removed U1: LM74930QRGERQ1, PB100:VQFN-24_RGE_4x4mm_P0.5mm_EP2.4mm, symbol PB100:PB100_LM74930QRGERQ1
- removed U2: INA228_Q1_PRELIM, symbol PB100:PB100_INA228_Q1_PRELIM
- added C20: 100nF 50V X7R DIFF, PB100:C0603, symbol PB100Gen:PB100G_C20
- added C21: 1nF 100V C0G, PB100:C0603, symbol PB100Gen:PB100G_C21
- added C22: 100nF 16V X7R, PB100:C0603, symbol PB100Gen:PB100G_C22
- added C23: 1nF PB I2C INT FILTER DNP, PB100:C0603, symbol PB100Gen:PB100G_C23
- added C24: 10nF 50V X7R, PB100:C0603, symbol PB100Gen:PB100G_C24
- added CCAP1: 100nF 25V X7R, PB100:C0603, symbol PB100Gen:PB100G_CCAP1
- added CSN1: 1nF 100V C0G DNP, PB100:C0603, symbol PB100Gen:PB100G_CSN1
- added CSN2: 1nF 200V C0G DNP, PB100:C0603, symbol PB100Gen:PB100G_CSN2
- added CVS1: CGA6N3X7R2A225M230AE 2.2uF 100V X7R; Ceff>=1uF@56V, PB100:C1210, symbol PB100Gen:PB100G_CVS1
- added D1: SM8S33AHM3/I, PB100:DO-218AC_Vishay_SM8S, symbol PB100Gen:PB100G_D1
- added DZVS1: 56V AUTOMOTIVE ZENER, PB100:SOD-123F, symbol PB100Gen:PB100G_DZVS1
- added J1: INPUT_CONNECTOR_CLASS_PRELIM (OFF-BOARD), symbol PB100Gen:PB100G_J1
- added JIN1: 40A PCB PIGTAIL TO NEAR-BATTERY 50A FUSE, PB100:POWER_PIGTAIL_2xTH_40A, symbol PB100Gen:PB100G_JIN1
- added JISO1: EVT INPUT-STAGE ISOLATION LINK — FITTED FOR NORMA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, PB100:EVT_INPUT_ISOLATION_LINK_M4, symbol PB100Gen:PB100G_JISO1
- added Q1: IAUT300N08S5N012ATMA2, PB100:PG-HSOF-8-1_TOLL_Infineon, symbol PB100Gen:PB100G_Q1
- added Q2: IAUTN15S6N025ATMA1, PB100:PG-HSOF-8-1_TOLL_Infineon, symbol PB100Gen:PB100G_Q2
- added R20: 10R 0.1% SHUNT FILTER, PB100:R0603, symbol PB100Gen:PB100G_R20
- added R21: 10R 0.1% SHUNT FILTER, PB100:R0603, symbol PB100Gen:PB100G_R21
- added R22: 1k 1% VBUS FILTER, PB100:R0603, symbol PB100Gen:PB100G_R22
- added R23: 10k PB I2C SDA PULL DNP, PB100:R0603, symbol PB100Gen:PB100G_R23
- added R24: 10k PB I2C SCL PULL DNP, PB100:R0603, symbol PB100Gen:PB100G_R24
- added R25: 47k PB I2C INT PULL DNP, PB100:R0603, symbol PB100Gen:PB100G_R25
- added R26: 0R INPUT FAULT AGGREGATE, PB100:R0603, symbol PB100Gen:PB100G_R26
- added R27: 200k 0.1% 100V, PB100:R0603, symbol PB100Gen:PB100G_R27
- added R28: 10k 0.1%, PB100:R0603, symbol PB100Gen:PB100G_R28
- added R29: 1k 0.1%, PB100:R0603, symbol PB100Gen:PB100G_R29
- added R3: 42.2k 1%, PB100:R0603, symbol PB100Gen:PB100G_R3
- added R4: 42.2k 1%, PB100:R0603, symbol PB100Gen:PB100G_R4
- added R5: 1.00k 1%, PB100:R0603, symbol PB100Gen:PB100G_R5
- added R6: 10k 1%, PB100:R0603, symbol PB100Gen:PB100G_R6
- added R7: 0R REPLACEABLE Q1 GATE, PB100:R0603, symbol PB100Gen:PB100G_R7
- added R8: 0R REPLACEABLE Q2 GATE, PB100:R0603, symbol PB100Gen:PB100G_R8
- added RSH1: CSS4J-4026R-L500F 0.5mR 5W FOUR-TERMINAL, PB100:CSS4J-4026_Bourns, symbol PB100Gen:PB100G_RSH1
- added RSN1: 100R DNP Q1 DAMPING, PB100:R0603, symbol PB100Gen:PB100G_RSN1
- added RSN2: 100R DNP Q2 DAMPING, PB100:R0603, symbol PB100Gen:PB100G_RSN2
- added TP001: TEST GND, PB100:TestPoint_SMD_1.5mm, symbol PB100Gen:PB100G_TP001
- added TP003: TEST VBAT_RAW, PB100:TestPoint_SMD_1.5mm, symbol PB100Gen:PB100G_TP003
- added TP004: TEST VBAT_REV_PROT, PB100:TestPoint_SMD_1.5mm, symbol PB100Gen:PB100G_TP004
- added TP005: TEST VBAT_PROT, PB100:TestPoint_SMD_1.5mm, symbol PB100Gen:PB100G_TP005
- added TP006: TEST IIN_SHUNT_HI, PB100:TestPoint_SMD_1.5mm, symbol PB100Gen:PB100G_TP006
- added TP007: TEST IIN_SHUNT_LO, PB100:TestPoint_SMD_1.5mm, symbol PB100Gen:PB100G_TP007
- added TP008: TEST VBAT_SENSE, PB100:TestPoint_SMD_1.5mm, symbol PB100Gen:PB100G_TP008
- added TP009: TEST IIN_SENSE, PB100:TestPoint_SMD_1.5mm, symbol PB100Gen:PB100G_TP009
- added TP062: TEST Q1_GATE, PB100:TestPoint_SMD_1.5mm, symbol PB100Gen:PB100G_TP062
- added TP063: TEST Q2_GATE, PB100:TestPoint_SMD_1.5mm, symbol PB100Gen:PB100G_TP063
- added TP064: TEST INPUT_COMMON_SOURCE, PB100:TestPoint_SMD_1.5mm, symbol PB100Gen:PB100G_TP064
- added TP065: TEST VBAT_PROT_PRELINK, PB100:TestPoint_SMD_1.5mm, symbol PB100Gen:PB100G_TP065
- added U1: LM74930QRGERQ1, PB100:VQFN-24_RGE_4x4mm_P0.5mm_EP2.4mm, symbol PB100Gen:PB100G_U1
- added U2: INA228AQDGSRQ1 TOTAL CURRENT MONITOR, PB100:VSSOP-10_L3.0-W3.0-P0.50-LS4.9-BL, symbol PB100Gen:PB100G_U2
Connections:
- net GND: now also C21.2, C22.2, C23.2, C24.2, CVS1.2, D1.2 (A), DZVS1.2, J1.2 (GND), JIN1.2 (GND), R28.2, R5.2, TP001.1 (GND), U1.11 (ILIM), U1.13 (GND), U1.16 (OVCLAMP), U1.9 (TMR), U2.1 (A1), U2.2 (A0), U2.7 (GND)
- net INPUT_COMMON_SOURCE: now also CSN1.2, CSN2.2, Q1.2 (S), Q1.3 (S), Q1.4 (S), Q1.5 (S), Q1.6 (S), Q1.7 (S), Q1.8 (S), Q2.2 (S), Q2.3 (S), Q2.4 (S), Q2.5 (S), Q2.6 (S), Q2.7 (S), Q2.8 (S), TP064.1 (INPUT_COMMON_SOURCE), U1.15 (OUT), U1.2 (A)
- net INPUT_PROT_FAULT_N: now also R26.1, U1.12 (FLT)
- net LM74930_CAP: now also CCAP1.1, U1.23 (CAP)
- net LM74930_OV: now also R4.2, R5.1, U1.5 (OV)
- net LM74930_OV_TOP_MID: now also R3.2, R4.1
- net LM74930_VS: now also CCAP1.2, CVS1.1, DZVS1.1, R6.2, U1.22 (VS), U1.4 (UVLO), U1.6 (EN), U1.7 (MODE)
- net PB_5V_OUT: now also C22.1, U2.6 (VS)
- net PB_I2C_INT: now also C23.1, R25.2, U2.3 (ALERT)
- net PB_I2C_SCL: now also R24.2, U2.5 (SCL)
- net PB_I2C_SDA: now also R23.2, U2.4 (SDA)
- net Q1_DGATE: now also R7.1, U1.1 (DGATE)
- net Q2_HGATE: now also R8.1, U1.14 (HGATE)
- net VBAT_PROT: now also JISO1.2 (BOARD_LOADS), R22.1, R27.1, TP005.1 (VBAT_PROT)
- net VBAT_RAW: now also D1.1 (K), J1.1 (VBAT_RAW), JIN1.1 (VBAT_RAW), Q2.Tab (D), R3.1, R6.1, RSN2.1, TP003.1 (VBAT_RAW)
- net VBAT_REV_PROT: now also Q1.Tab (D), RSH1.1 (PWR_IN), RSN1.1, TP004.1 (VBAT_REV_PROT), U1.18 (ISCP), U1.19 (CS-), U1.20 (CS+), U1.24 (C)
- new net IIN_MON_N: C20.2, R21.2, U2.9 (IN-)
- new net IIN_MON_P: C20.1, R20.2, U2.10 (IN+)
- new net IIN_SENSE: TP009.1 (IIN_SENSE)
- new net IIN_SHUNT_HI: R20.1, RSH1.3 (SNS_IN), TP006.1 (IIN_SHUNT_HI)
- new net IIN_SHUNT_LO: R21.1, RSH1.4 (SNS_OUT), TP007.1 (IIN_SHUNT_LO)
- new net IIN_VBUS_FILTERED: C21.1, R22.2, U2.8 (VBUS)
- new net LB_3V3_IO: R23.1, R24.1, R25.1
- new net PB_FAULT: R26.2
- new net Q1_GATE: Q1.1 (G), R7.2, TP062.1 (Q1_GATE)
- new net Q1_SNUB: CSN1.1, RSN1.2
- new net Q2_GATE: Q2.1 (G), R8.2, TP063.1 (Q2_GATE)
- new net Q2_SNUB: CSN2.1, RSN2.2
- new net VBAT_PROT_PRELINK: JISO1.1 (INPUT_STAGE), RSH1.2 (PWR_OUT), TP065.1 (VBAT_PROT_PRELINK)
- new net VBAT_SENSE: C24.1, R29.2, TP008.1 (VBAT_SENSE)
- new net VBAT_SENSE_RAW: R27.2, R28.1, R29.1
Other:
- note added: "Work queue: CAP-INP. ADR-0018/0019/0020 implementation. The raw-side 150 V Q2 and protected-side 80 V Q1 retain the reviewed LM74930-Q1 common-source hard-cutoff topology. RSH1 is a 0.5 mOhm four-terminal shunt. JISO1 is the mandatory removable input-stage isolation link; opening it prevents VBAT_PROT from energizing the remainder of the board. D1 is a legacy DNP comparison site and is never cred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"
- note removed: "Input protection capture notes: - ADR-0018 selects LM74930-Q1 hard cutoff and permits load disconnection during load dump - Q2 IAUTN15S6N025ATMA1 150 V is the raw-side HGATE cutoff FET - Q1 IAUT300N08S5N012ATMA2 80 V is the protected DGATE reverse FET - R3/R4/R5 42.2k+42.2k/1.00k 1% set a generated 48.99-54.89 V cutoff - D1 SM8S33AHM3/I is DNP legacy footprint only and is not an approved energy s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"
- title: PB-100 Input Protection -> PB-100 Input Protection and Total-Current Monitor — Rev.1 EVT
