File: hardware/power-board/PB-100/kicad/sheets/telemetry.kicad_sch (KiCad schematic)
At the start: 4 parts

Commit message: Add PB-100 current telemetry derivation precheck
Other:
- note added: "Telemetry capture notes: - Source traces: PB-100-current-telemetry-trace.csv, PB-100-current-telemetry-freeze-review.csv, PB-100-current-telemetry-value-freeze-checklist.csv, PB-100-current-telemetry-value-derivation-precheck.csv, PB-100-thermal-telemetry-trace.csv, PB-100-thermal-telemetry-freeze-review.csv, PB-100-thermal-telemetry-value-freeze-checklist.csv - Thermal nets TEMP_PCB, TEMP_PWR_A,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"
- note removed: "Telemetry capture notes: - Source traces: PB-100-current-telemetry-trace.csv, PB-100-current-telemetry-freeze-review.csv, PB-100-current-telemetry-value-freeze-checklist.csv, PB-100-thermal-telemetry-trace.csv, PB-100-thermal-telemetry-freeze-review.csv, PB-100-thermal-telemetry-value-freeze-checklist.csv - Thermal nets TEMP_PCB, TEMP_PWR_A, TEMP_PWR_B map to LB-100 telemetry - Board ID stays sep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"
Changed lines of the file:
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@@
     (comment 9 "Work queue: CAP-TEL. Preliminary schematic capture follows PB-100-schematic-capture-work-queue.csv.")
     (comment 1 "Preliminary capture for current, voltage, thermal, and board ID telemetry.")
-    (comment 2 "Sources: PB-100-current-telemetry-trace.csv, PB-100-current-telemetry-freeze-review.csv, PB-100-current-telemetry-value-freeze-checklist.csv, PB-100-thermal-telemetry-trace.csv, PB-100-thermal-telemetry-freeze-review.csv, PB-100-thermal-telemetry-value-freeze-checklist.csv, telemetry maps.")
+    (comment 2 "Sources: PB-100-current-telemetry-trace.csv, PB-100-current-telemetry-freeze-review.csv, PB-100-current-telemetry-value-freeze-checklist.csv, PB-100-current-telemetry-value-derivation-precheck.csv, PB-100-thermal-telemetry-trace.csv, PB-100-thermal-telemetry-freeze-review.csv, PB-100-thermal-telemetry-value-freeze-checklist.csv, telemetry maps.")
   )
-  (text "Telemetry capture notes:\n- Source traces: PB-100-current-telemetry-trace.csv, PB-100-current-telemetry-freeze-review.csv, PB-100-current-telemetry-value-freeze-checklist.csv, PB-100-thermal-telemetry-trace.csv, PB-100-thermal-telemetry-freeze-review.csv, PB-100-thermal-telemetry-value-freeze-checklist.csv\n- Thermal nets TEMP_PCB, TEMP_PWR_A, TEMP_PWR_B map to LB-100 telemetry\n- Board ID stays separate from vehicle role mapping\n\nNo PCB layout from this preliminary capture."
+  (text "Telemetry capture notes:\n- Source traces: PB-100-current-telemetry-trace.csv, PB-100-current-telemetry-freeze-review.csv, PB-100-current-telemetry-value-freeze-checklist.csv, PB-100-current-telemetry-value-derivation-precheck.csv, PB-100-thermal-telemetry-trace.csv, PB-100-thermal-telemetry-freeze-review.csv, PB-100-thermal-telemetry-value-freeze-checklist.csv\n- Thermal nets TEMP_PCB, TEMP_PWR_A, TEMP_PWR_B map to LB-100 telemetry\n- Board ID stays separate from vehicle role mapping\n\nNo PCB layout from this preliminary capture."
     (at 20 20 0)
     (effects (font (size 2.0 2.0)) (justify left top))
