File: hardware/power-board/PB-100/kicad/sheets/telemetry.kicad_sch (KiCad schematic)
At the start: 4 parts

Commit message: Advance PB-100 EVT routing baseline
Parts:
- removed RID1: BOARD_ID_RESISTOR_CLASS_PRELIM, symbol PB100:PB100_BOARD_ID_RESISTOR_CLASS_PRELIM
- removed RT1, RT2, RT3: THERMAL_NTC_PRELIM, symbol PB100:PB100_THERMAL_NTC_PRELIM
- added C61: 10nF 50V X7R, PB100:C0603, symbol PB100Gen:PB100G_C61
- added C64: 10nF 50V X7R, PB100:C0603, symbol PB100Gen:PB100G_C64
- added C67: 10nF 50V X7R, PB100:C0603, symbol PB100Gen:PB100G_C67
- added R61: 4.7k 1% AEC-Q200, PB100:R0603, symbol PB100Gen:PB100G_R61
- added R62: 1k 1% ADC SERIES, PB100:R0603, symbol PB100Gen:PB100G_R62
- added R64: 4.7k 1% AEC-Q200, PB100:R0603, symbol PB100Gen:PB100G_R64
- added R65: 1k 1% ADC SERIES, PB100:R0603, symbol PB100Gen:PB100G_R65
- added R67: 4.7k 1% AEC-Q200, PB100:R0603, symbol PB100Gen:PB100G_R67
- added R68: 1k 1% ADC SERIES, PB100:R0603, symbol PB100Gen:PB100G_R68
- added RID1: PB REV1 ID: 10k/10k 0.1% DIVIDER, PB100:Board_ID_Divider_0603x2, symbol PB100Gen:PB100G_RID1
- added RT1: NTCGS103JF103FT8 10k 1% B3435 AEC-Q200, PB100:R0402, symbol PB100Gen:PB100G_RT1
- added RT2: NTCGS103JF103FT8 10k 1% B3435 AEC-Q200, PB100:R0402, symbol PB100Gen:PB100G_RT2
- added RT3: NTCGS103JF103FT8 10k 1% B3435 AEC-Q200, PB100:R0402, symbol PB100Gen:PB100G_RT3
- added TP002: TEST AGND, PB100:TestPoint_SMD_1.5mm, symbol PB100Gen:PB100G_TP002
- added TP012: TEST LB_3V3_IO, PB100:TestPoint_SMD_1.5mm, symbol PB100Gen:PB100G_TP012
- added TP013: TEST PB_I2C_SCL, PB100:TestPoint_SMD_1.5mm, symbol PB100Gen:PB100G_TP013
- added TP014: TEST PB_I2C_SDA, PB100:TestPoint_SMD_1.5mm, symbol PB100Gen:PB100G_TP014
- added TP015: TEST PB_I2C_INT, PB100:TestPoint_SMD_1.5mm, symbol PB100Gen:PB100G_TP015
- added TP016: TEST TEMP_PCB, PB100:TestPoint_SMD_1.5mm, symbol PB100Gen:PB100G_TP016
- added TP017: TEST TEMP_PWR_A, PB100:TestPoint_SMD_1.5mm, symbol PB100Gen:PB100G_TP017
- added TP018: TEST TEMP_PWR_B, PB100:TestPoint_SMD_1.5mm, symbol PB100Gen:PB100G_TP018
- added TP019: TEST CAN1_TX_DISABLE_CMD, PB100:TestPoint_SMD_1.5mm, symbol PB100Gen:PB100G_TP019
- added TP020: TEST CAN1_TX_DISABLED_STATUS, PB100:TestPoint_SMD_1.5mm, symbol PB100Gen:PB100G_TP020
- added TP021: TEST CAN1_RX_ROUTE, PB100:TestPoint_SMD_1.5mm, symbol PB100Gen:PB100G_TP021
Connections:
- net GND: now also C61.2, C64.2, C67.2, RID1.3 (GND), RT1.2, RT2.2, RT3.2
- net LB_3V3_IO: now also R61.1, R64.1, R67.1, RID1.1 (LB_3V3_IO), TP012.1 (LB_3V3_IO)
- net PB_ID_ADC: now also RID1.2 (PB_ID_ADC)
- net TEMP_PCB: now also C61.1, R62.2, TP016.1 (TEMP_PCB)
- net TEMP_PWR_A: now also C64.1, R65.2, TP017.1 (TEMP_PWR_A)
- net TEMP_PWR_B: now also C67.1, R68.2, TP018.1 (TEMP_PWR_B)
- new net AGND: TP002.1 (AGND)
- new net CAN1_RX_ROUTE: TP021.1 (CAN1_RX_ROUTE)
- new net CAN1_TX_DISABLED_STATUS: TP020.1 (CAN1_TX_DISABLED_STATUS)
- new net CAN1_TX_DISABLE_CMD: TP019.1 (CAN1_TX_DISABLE_CMD)
- new net PB_I2C_INT: TP015.1 (PB_I2C_INT)
- new net PB_I2C_SCL: TP013.1 (PB_I2C_SCL)
- new net PB_I2C_SDA: TP014.1 (PB_I2C_SDA)
- new net TEMP_PCB_RAW: R61.2, R62.1, RT1.1
- new net TEMP_PWR_A_RAW: R64.2, R65.1, RT2.1
- new net TEMP_PWR_B_RAW: R67.2, R68.1, RT3.1
Other:
- note added: "Work queue: CAP-TEL. Three role-independent 10k AEC-Q200 NTC dividers use 4.7k pull-ups to LB_3V3_IO, 1k ADC isolation, and 10nF filters. Sensor placement targets board reference, input/OUT2 hot zone, and medium-output/buck zone. RID1 is a physical two-resistor board-ID divider. Calibration and thresholds remain configuration-owned and require EVT measurement."
- note removed: "Telemetry capture notes: - Source traces: PB-100-current-telemetry-trace.csv, PB-100-current-telemetry-freeze-review.csv, PB-100-current-telemetry-value-freeze-checklist.csv, PB-100-current-telemetry-value-derivation-precheck.csv, PB-100-current-telemetry-closeout-precheck.csv, PB-100-thermal-telemetry-trace.csv, PB-100-thermal-telemetry-freeze-review.csv, PB-100-thermal-telemetry-value-freeze-ch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"
- title: PB-100 Telemetry -> PB-100 Thermal and Board-Identity Telemetry — Rev.1 EVT
