File: hardware/power-board/PB-100/kicad/sheets/logic-power.kicad_sch (KiCad schematic)
At the start: 2 parts, among them U3 LM5164QDDATQ1_PRELIM

Commit message: Advance PB-100 EVT routing baseline
Parts:
- removed L1: BUCK_INDUCTOR_CLASS_PRELIM, symbol PB100:PB100_BUCK_INDUCTOR_CLASS_PRELIM
- removed U3: LM5164QDDATQ1_PRELIM, symbol PB100:PB100_LM5164QDDATQ1_PRELIM
- added C30: 2.2uF 100V X7R, PB100:C1210, symbol PB100Gen:PB100G_C30
- added C31: 100nF 100V X7R, PB100:C0805, symbol PB100Gen:PB100G_C31
- added C32: 10uF 100V BULK CANDIDATE, PB100:C1210, symbol PB100Gen:PB100G_C32
- added C33: 2.2nF 50V X7R, PB100:C0603, symbol PB100Gen:PB100G_C33
- added C34: 22uF 10V X7R, PB100:C1210, symbol PB100Gen:PB100G_C34
- added C35: 22uF 10V X7R, PB100:C1210, symbol PB100Gen:PB100G_C35
- added C36: 100nF 16V X7R, PB100:C0603, symbol PB100Gen:PB100G_C36
- added C37: 10nF PGOOD FILTER DNP, PB100:C0603, symbol PB100Gen:PB100G_C37
- added C38: 3.3nF 100V C0G TYPE3 CA, PB100:C0603, symbol PB100Gen:PB100G_C38
- added C39: 180pF 50V C0G TYPE3 CB, PB100:C0603, symbol PB100Gen:PB100G_C39
- added C40: 1nF 100V C0G DNP, PB100:C0603, symbol PB100Gen:PB100G_C40
- added L1: 47uH SHIELDED AEC-Q200; Isat>=2.2A Irms>=1.2A, PB100:Inductor_12x12mm, symbol PB100Gen:PB100G_L1
- added R30: 332k 1%, PB100:R0603, symbol PB100Gen:PB100G_R30
- added R31: 100k 1%, PB100:R0603, symbol PB100Gen:PB100G_R31
- added R32: 41.2k 1%, PB100:R0603, symbol PB100Gen:PB100G_R32
- added R33: 158k 0.1%, PB100:R0603, symbol PB100Gen:PB100G_R33
- added R34: 49.9k 0.1%, PB100:R0603, symbol PB100Gen:PB100G_R34
- added R35: 47k PGOOD PULL-UP, PB100:R0603, symbol PB100Gen:PB100G_R35
- added R36: 110k 1% TYPE3 RA, PB100:R0603, symbol PB100Gen:PB100G_R36
- added R37: 100R BUCK SNUBBER DNP, PB100:R0603, symbol PB100Gen:PB100G_R37
- added TP010: TEST PB_5V_OUT, PB100:TestPoint_SMD_1.5mm, symbol PB100Gen:PB100G_TP010
- added TP011: TEST PB_PWR_GOOD, PB100:TestPoint_SMD_1.5mm, symbol PB100Gen:PB100G_TP011
- added U3: LM5164QDDATQ1 100V 1A BUCK, PB100:SOIC-8_L4.9-W3.9-P1.27-LS6.0-BL-EP2.9, symbol PB100Gen:PB100G_U3
Connections:
- net GND: now also C30.2, C31.2, C32.2, C34.2, C35.2, C36.2, C37.2, C40.2, R31.2, R32.2, R34.2, U3.1 (GND), U3.9 (EP)
- net PB_5V_OUT: now also C34.1, C35.1, C36.1, L1.2, R33.1, R36.2, TP010.1 (PB_5V_OUT)
- net PB_PWR_GOOD: now also C37.1, R35.2, TP011.1 (PB_PWR_GOOD), U3.6 (PGOOD)
- net VBAT_PROT: now also C30.1, C31.1, C32.1, R30.1, U3.2 (VIN)
- new net BUCK_BST: C33.1, U3.7 (BST)
- new net BUCK_EN_UVLO: R30.2, R31.1, U3.3 (EN/UVLO)
- new net BUCK_FB: C39.2, R33.2, R34.1, U3.5 (FB)
- new net BUCK_RAMP: C38.2, C39.1, R36.1
- new net BUCK_RON_SET: R32.1, U3.4 (RON)
- new net BUCK_SNUB: C40.1, R37.2
- new net BUCK_SW: C33.2, C38.1, L1.1, R37.1, U3.8 (SW)
- new net LB_3V3_IO: R35.1
Other:
- note added: "Work queue: CAP-LOGIC. LM5164-Q1 100 V synchronous buck, 5.0 V / 1 A planning limit. The 300 kHz candidate uses 41.2k RON, 47uH shielded inductor, and a type-3 ripple-injection network. Switch-node copper must remain compact; thermal vias under the exposed pad and routed EMI evidence are required at EVT-FAB-REVIEW. PB_5V_OUT never powers accessory loads."
- note removed: "Logic power capture notes: - Source trace: PB-100-logic-power-rail-trace.csv - Freeze review: PB-100-logic-power-freeze-review.csv - Value freeze checklist: PB-100-logic-power-value-freeze-checklist.csv - Value derivation precheck: PB-100-logic-power-value-derivation-precheck.csv - Closeout precheck: PB-100-logic-power-closeout-precheck.csv - U3 LM5164-Q1-class preferred buck - LM5013-Q1-class hi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"
- title: PB-100 Logic Power -> PB-100 Protected 5 V Logic Supply — Rev.1 EVT
