File: hardware/logic-board/LB-100/kicad/LB-100.kicad_sch (KiCad schematic)
At the start: 0 parts

Commit message: Close LB FB schematic freeze
Other:
- note added: "Reviewed LB-100 value-bearing schematic inputs: - MCU baseline STM32H563VITx LQFP100; STM32H573VITx security alternate; STM32H563RGT6 fallback only after resource reduction. - PB_5V_OUT budget: 500 mA sustained allocation; 219.2 mA sustained LB load; 415.2 mA service peak; USB no-back-power boundary. - JPB1: exact OUT1_CTL..OUT10_CTL, OUT1_FLT..OUT10_FLT, OUT1_IMON..OUT10_IMON, PB_I2C, CAN1, CAN2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"
- note added: "Schematic freeze evidence: - ../LB-100-schematic-review-closeout.md - ../LB-100-stm32h563-pin-binding-precheck.csv - ../LB-100-rail-budget-closeout-precheck.csv - ../LB-100-communication-safety-precheck.csv - ../LB-100-service-storage-sensor-precheck.csv - ../LB-100-mcu-sourcing-precheck.csv - ../LB-100-component-sourcing-precheck.csv PCB layout and manufacturing outputs remain separate post-free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"
Changed lines of the file:
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@@
+    )
+  )
+  (text "Reviewed LB-100 value-bearing schematic inputs:\n- MCU baseline STM32H563VITx LQFP100; STM32H573VITx security alternate; STM32H563RGT6 fallback only after resource reduction.\n- PB_5V_OUT budget: 500 mA sustained allocation; 219.2 mA sustained LB load; 415.2 mA service peak; USB no-back-power boundary.\n- JPB1: exact OUT1_CTL..OUT10_CTL, OUT1_FLT..OUT10_FLT, OUT1_IMON..OUT10_IMON, PB_I2C, CAN1, CAN2, LIN/RS485/UART, and spare binding per LB-100-stm32h563-pin-binding-precheck.csv.\n- CAN1: DNP/open TX route; read-only default; no firmware-only vehicle-CAN TX enable.\n- Services: USB service, BLE, microSD, RTC, FRAM, IMU, lux, SWD, BOOT0, reset, service button."
+    (at 155 35 0)
+    (effects
+      (font
+        (size 1.6 1.6)
+      )
+      (justify left top)
+    )
+  )
+  (text "Schematic freeze evidence:\n- ../LB-100-schematic-review-closeout.md\n- ../LB-100-stm32h563-pin-binding-precheck.csv\n- ../LB-100-rail-budget-closeout-precheck.csv\n- ../LB-100-communication-safety-precheck.csv\n- ../LB-100-service-storage-sensor-precheck.csv\n- ../LB-100-mcu-sourcing-precheck.csv\n- ../LB-100-component-sourcing-precheck.csv\n\nPCB layout and manufacturing outputs remain separate post-freeze work."
+    (at 155 130 0)
+    (effects
+      (font
+        (size 1.6 1.6)
+      )
+      (justify left top)
     )
   )

Commit message: Add three-board footprint binding inventory
Other:
- note added: "Blocked in this scaffold: - KiCad board import while footprint binding is open - KiCad board import while mechanical envelope is open - Gerber generation - drill files - pick-place files - BOM/CPL order package - vehicle-CAN TX enable path"
- note added: "LB-100 schematic scaffold only. Do not create LB-100.kicad_pcb from this project until ../LB-100-pcb-layout-start-checklist.csv closes footprint binding and mechanical envelope gates. Primary inputs: - ../LB-100-requirements.md - ../LB-100-power-budget-precheck.md - ../LB-100-schematic-freeze-checklist.md - ../LB-100-pcb-layout-start-checklist.csv - ../LB-100-footprint-binding-inventory.csv - ../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"
- note added: "Schematic freeze evidence: - ../LB-100-schematic-review-closeout.md - ../LB-100-stm32h563-pin-binding-precheck.csv - ../LB-100-rail-budget-closeout-precheck.csv - ../LB-100-communication-safety-precheck.csv - ../LB-100-service-storage-sensor-precheck.csv - ../LB-100-mcu-sourcing-precheck.csv - ../LB-100-component-sourcing-precheck.csv - ../LB-100-pcb-layout-start-checklist.csv - ../LB-100-footpri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"
- note removed: "Blocked in this scaffold: - PCB layout - Gerber generation - drill files - pick-place files - BOM/CPL order package - vehicle-CAN TX enable path"
- note removed: "LB-100 schematic scaffold only. Do not create PCB layout from this project until LB-100 schematic freeze is closed. Primary inputs: - ../LB-100-requirements.md - ../LB-100-power-budget-precheck.md - ../LB-100-schematic-freeze-checklist.md - ../LB-100-board-release-blocker-register.csv - ../../../power-board/PB-100/PB-100-b2b-pin-map.csv"
- note removed: "Schematic freeze evidence: - ../LB-100-schematic-review-closeout.md - ../LB-100-stm32h563-pin-binding-precheck.csv - ../LB-100-rail-budget-closeout-precheck.csv - ../LB-100-communication-safety-precheck.csv - ../LB-100-service-storage-sensor-precheck.csv - ../LB-100-mcu-sourcing-precheck.csv - ../LB-100-component-sourcing-precheck.csv PCB layout and manufacturing outputs remain separate post-free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"
Changed lines of the file:
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@@
     (rev "schematic-scaffold")
     (company "SVC Platform")
-    (comment 1 "Schematic scaffold only. PCB layout is blocked until LB-100 schematic freeze.")
+    (comment 1 "Schematic freeze closed. Board import is blocked by layout-start gates.")
     (comment 2 "Requirements: ../LB-100-requirements.md and ADR-0014.")
     (comment 3 "CAN1 vehicle interface remains read-only by default.")
     (comment 4 "PB_5V_OUT allocation is 500 mA sustained unless reviewed.")
   )
-  (text "LB-100 schematic scaffold only.\n\nDo not create PCB layout from this project until LB-100 schematic freeze is closed.\n\nPrimary inputs:\n- ../LB-100-requirements.md\n- ../LB-100-power-budget-precheck.md\n- ../LB-100-schematic-freeze-checklist.md\n- ../LB-100-board-release-blocker-register.csv\n- ../../../power-board/PB-100/PB-100-b2b-pin-map.csv"
+  (text "LB-100 schematic scaffold only.\n\nDo not create LB-100.kicad_pcb from this project until ../LB-100-pcb-layout-start-checklist.csv closes footprint binding and mechanical envelope gates.\n\nPrimary inputs:\n- ../LB-100-requirements.md\n- ../LB-100-power-budget-precheck.md\n- ../LB-100-schematic-freeze-checklist.md\n- ../LB-100-pcb-layout-start-checklist.csv\n- ../LB-100-footprint-binding-inventory.csv\n- ../LB-100-board-release-blocker-register.csv\n- ../../../power-board/PB-100/PB-100-b2b-pin-map.csv"
     (at 30 35 0)
     (effects
@@
     )
   )
-  (text "Blocked in this scaffold:\n- PCB layout\n- Gerber generation\n- drill files\n- pick-place files\n- BOM/CPL order package\n- vehicle-CAN TX enable path"
+  (text "Blocked in this scaffold:\n- KiCad board import while footprint binding is open\n- KiCad board import while mechanical envelope is open\n- Gerber generation\n- drill files\n- pick-place files\n- BOM/CPL order package\n- vehicle-CAN TX enable path"
     (at 30 105 0)
     (effects
@@
     )
   )
-  (text "Schematic freeze evidence:\n- ../LB-100-schematic-review-closeout.md\n- ../LB-100-stm32h563-pin-binding-precheck.csv\n- ../LB-100-rail-budget-closeout-precheck.csv\n- ../LB-100-communication-safety-precheck.csv\n- ../LB-100-service-storage-sensor-precheck.csv\n- ../LB-100-mcu-sourcing-precheck.csv\n- ../LB-100-component-sourcing-precheck.csv\n\nPCB layout and manufacturing outputs remain separate post-freeze work."
+  (text "Schematic freeze evidence:\n- ../LB-100-schematic-review-closeout.md\n- ../LB-100-stm32h563-pin-binding-precheck.csv\n- ../LB-100-rail-budget-closeout-precheck.csv\n- ../LB-100-communication-safety-precheck.csv\n- ../LB-100-service-storage-sensor-precheck.csv\n- ../LB-100-mcu-sourcing-precheck.csv\n- ../LB-100-component-sourcing-precheck.csv\n- ../LB-100-pcb-layout-start-checklist.csv\n- ../LB-100-footprint-binding-inventory.csv\n\nPCB layout and manufacturing outputs remain separate post-freeze work."
     (at 155 130 0)
     (effects
