File: hardware/logic-board/LB-100/kicad/LB-100.kicad_sch (KiCad schematic)
At the start: 0 parts

Commit message: feat(hardware): close LB FB schematics and FX18 mechanics
Parts:
- added C1: 1uF 10V X7R, LB100:R_C_0603_1608Metric, symbol LB100:LB100_C1
- added C10: 18pF 50V C0G, LB100:R_C_0603_1608Metric, symbol LB100:LB100_C10
- added C11: 8.2pF 50V C0G, LB100:R_C_0603_1608Metric, symbol LB100:LB100_C11
- added C12: 8.2pF 50V C0G, LB100:R_C_0603_1608Metric, symbol LB100:LB100_C12
- added C13: 1nF 50V C0G, LB100:R_C_0603_1608Metric, symbol LB100:LB100_C13
- added C14: 1nF 50V C0G, LB100:R_C_0603_1608Metric, symbol LB100:LB100_C14
- added C15: 100nF 6.3V X7R, LB100:R_C_0603_1608Metric, symbol LB100:LB100_C15
- added C16: 100nF 6.3V X7R, LB100:R_C_0603_1608Metric, symbol LB100:LB100_C16
- added C17: 100nF 6.3V X7R, LB100:R_C_0603_1608Metric, symbol LB100:LB100_C17
- added C18: 100nF 6.3V X7R, LB100:R_C_0603_1608Metric, symbol LB100:LB100_C18
- added C19: 100nF 6.3V X7R, LB100:R_C_0603_1608Metric, symbol LB100:LB100_C19
- added C2: 1uF 6.3V X7R, LB100:R_C_0603_1608Metric, symbol LB100:LB100_C2
- added C20: 100nF 6.3V X7R, LB100:R_C_0603_1608Metric, symbol LB100:LB100_C20
- added C21: 100nF 6.3V X7R, LB100:R_C_0603_1608Metric, symbol LB100:LB100_C21
- added C22: 100nF 6.3V X7R, LB100:R_C_0603_1608Metric, symbol LB100:LB100_C22
- added C23: 100nF 6.3V X7R, LB100:R_C_0603_1608Metric, symbol LB100:LB100_C23
- added C24: 100nF 6.3V X7R, LB100:R_C_0603_1608Metric, symbol LB100:LB100_C24
- added C25: 100nF 6.3V X7R, LB100:R_C_0603_1608Metric, symbol LB100:LB100_C25
- added C26: 100nF 6.3V X7R, LB100:R_C_0603_1608Metric, symbol LB100:LB100_C26
- added C27: 100nF 6.3V X7R, LB100:R_C_0603_1608Metric, symbol LB100:LB100_C27
- added C3: 10uF 6.3V X7R, LB100:R_C_0805_2012Metric, symbol LB100:LB100_C3
- added C4: 1uF 6.3V X7R, LB100:R_C_0603_1608Metric, symbol LB100:LB100_C4
- added C5: 100nF 6.3V X7R, LB100:R_C_0603_1608Metric, symbol LB100:LB100_C5
- added C6: 2.2uF 6.3V X7R, LB100:R_C_0603_1608Metric, symbol LB100:LB100_C6
- added C7: 2.2uF 6.3V X7R, LB100:R_C_0603_1608Metric, symbol LB100:LB100_C7
- added C8: 100nF 6.3V X7R, LB100:R_C_0603_1608Metric, symbol LB100:LB100_C8
- added C9: 18pF 50V C0G, LB100:R_C_0603_1608Metric, symbol LB100:LB100_C9
- added FB1: 600R@100MHz 0.2A, LB100:R_C_0603_1608Metric, symbol LB100:LB100_FB1
- added JBT1: BACKUP_BATTERY_2V3_TO_3V6_DNP, LB100:PinHeader_1x02_P2.54mm_Vertical, symbol LB100:LB100_JBT1
- added JDBG1: SWD_2x3_1.27mm, LB100:PinHeader_2x03_P1.27mm_Vertical, symbol LB100:LB100_JDBG1
- added JFB1: AFC07-S24ECA-00, LB100:FPC-SMD_AFC07-S24ECA-00, symbol LB100:LB100_JFB1
- added JPB1: FX18-100S-0.8SV10, LB100:FX18-100S-0.8SV10_Hirose, symbol LB100:LB100_JPB1
- added JSD1: TF-015, LB100:TF-SMD_TF-015, symbol LB100:LB100_JSD1
- added R1: 100k 1%, LB100:R_C_0603_1608Metric, symbol LB100:LB100_R1
- added R10: 47k 1%, LB100:R_C_0603_1608Metric, symbol LB100:LB100_R10
- added R11: 47k 1%, LB100:R_C_0603_1608Metric, symbol LB100:LB100_R11
- added R12: 10k 1%, LB100:R_C_0603_1608Metric, symbol LB100:LB100_R12
- added R13: 0R, LB100:R_C_0603_1608Metric, symbol LB100:LB100_R13
- added R14: 0R, LB100:R_C_0603_1608Metric, symbol LB100:LB100_R14
- added R15: 0R, LB100:R_C_0603_1608Metric, symbol LB100:LB100_R15
- added R2: 0R, LB100:R_C_0603_1608Metric, symbol LB100:LB100_R2
- added R3: 0R, LB100:R_C_0603_1608Metric, symbol LB100:LB100_R3
- added R4: 10k 1%, LB100:R_C_0603_1608Metric, symbol LB100:LB100_R4
- added R5: 10k 1%, LB100:R_C_0603_1608Metric, symbol LB100:LB100_R5
- added R6: 2.2k 1%, LB100:R_C_0603_1608Metric, symbol LB100:LB100_R6
- added R7: 2.2k 1%, LB100:R_C_0603_1608Metric, symbol LB100:LB100_R7
- added R8: 4.7k 1%, LB100:R_C_0603_1608Metric, symbol LB100:LB100_R8
- added R9: 10k 1%, LB100:R_C_0603_1608Metric, symbol LB100:LB100_R9
- added U1: STM32H563VIT6, LB100:LQFP-100_L14.0-W14.0-P0.50-LS16.0-BL, symbol LB100:LB100_U1
- added U10: BMI270, LB100:LGA-14_L3.0-W2.5-P0.50-BR, symbol LB100:LB100_U10
- added U11: VEML7700-TT, LB100:SENSOR-SMD_EML7700-TT, symbol LB100:LB100_U11
- added U12: TPS22918TDBVRQ1, LB100:SOT-23-6_L2.9-W1.6-P0.95-LS2.8-BL, symbol LB100:LB100_U12
- added U13: TPS22918TDBVRQ1, LB100:SOT-23-6_L2.9-W1.6-P0.95-LS2.8-BL, symbol LB100:LB100_U13
- added U2: XC6220B331MR-G, LB100:SOT-25_L3.0-W1.6-P0.95-LS2.8-TL, symbol LB100:LB100_U2
- added U3: TCA9539QPWRQ1, LB100:TSSOP-24_4.4x7.8mm_P0.65mm, symbol LB100:LB100_U3
- added U4: TJA1051TK/3,118, LB100:HVSON-8_L3.0-W3.0-P0.65-BL-EP, symbol LB100:LB100_U4
- added U5: TJA1021T/20/CM,118, LB100:SOIC-8_L4.9-W3.9-P1.27-LS6.0-BL, symbol LB100:LB100_U5
- added U6: SP3485EN-L/TR, LB100:SOIC-8_L5.0-W4.0-P1.27-LS6.0-BL, symbol LB100:LB100_U6
- added U7: E73-2G4M08S1C, LB100:WIRELM-SMD_E73-2G4M08S1C, symbol LB100:LB100_U7
- added U8: FM24CL64B-GTR, LB100:SOIC-8_L4.9-W3.9-P1.27-LS6.0-BL, symbol LB100:LB100_U8
- added U9: DS3231MZ+TRL, LB100:SOIC-8_L4.9-W3.9-P1.27-LS6.0-BL, symbol LB100:LB100_U9
- added Y1: ABM8AIG-25.000MHZ-12-2Z-T3, LB100:Crystal_SMD_3225-4Pin, symbol LB100:LB100_Y1
- added Y2: ABS07AIG-32.768kHz-7-T, LB100:Crystal_SMD_3215-2Pin, symbol LB100:LB100_Y2
Connections:
- new net ADC_REF: JPB1.66 (ADC_REF), U1.21 (VREF+)
- new net AGND: C4.2, C5.2, JPB1.11 (AGND), JPB1.12 (AGND), U1.19 (VSSA), U1.20 (VREF-)
- new net BACKUP_AON: JBT1.1 (BACKUP_AON), U9.6 (VBAT)
- new net BLE_RESET_N: R9.2, U1.97 (PE0), U7.26 (RESET)
- new net BOOT0: R5.1, U1.94 (BOOT0)
- new net CAN1_RX_ROUTE: JPB1.69 (CAN1_RX_ROUTE), U1.95 (PB8)
- new net CAN1_TX_DISABLED_STATUS: JPB1.68 (CAN1_TX_DISABLED_STATUS), U1.58 (PD11)
- new net CAN1_TX_DISABLE_CMD: JPB1.67 (CAN1_TX_DISABLE_CMD), U1.85 (PD4)
- new net CAN1_TX_ROUTE: JPB1.70 (CAN1_TX_ROUTE), U1.96 (PB9)
- new net CAN2_RX_ROUTE: JPB1.71 (CAN2_RX_ROUTE), U1.51 (PB12), U4.4 (RXD)
- new net CAN2_TX_ROUTE: JPB1.72 (CAN2_TX_ROUTE), U1.52 (PB13), U4.1 (TXD)
- new net CH_LED_1: JFB1.10 (CH_LED_1), U3.4 (P00)
- new net CH_LED_10: JFB1.19 (CH_LED_10), U3.14 (P11)
- new net CH_LED_2: JFB1.11 (CH_LED_2), U3.5 (P01)
- new net CH_LED_3: JFB1.12 (CH_LED_3), U3.6 (P02)
- new net CH_LED_4: JFB1.13 (CH_LED_4), U3.7 (P03)
- new net CH_LED_5: JFB1.14 (CH_LED_5), U3.8 (P04)
- new net CH_LED_6: JFB1.15 (CH_LED_6), U3.9 (P05)
- new net CH_LED_7: JFB1.16 (CH_LED_7), U3.10 (P06)
- new net CH_LED_8: JFB1.17 (CH_LED_8), U3.11 (P07)
- new net CH_LED_9: JFB1.18 (CH_LED_9), U3.13 (P10)
- new net EXT_5V_EN: JPB1.84 (EXT_5V_EN), U1.69 (PA10)
- new net EXT_ADC1: JPB1.80 (EXT_ADC1), U1.64 (PC7)
- new net EXT_ADC2: JPB1.81 (EXT_ADC2), U1.65 (PC8)
- new net EXT_DIG1: JPB1.82 (EXT_DIG1), U1.67 (PA8)
- new net EXT_DIG2: JPB1.83 (EXT_DIG2), U1.68 (PA9)
- new net FB_3V3_OR_IO: JFB1.2 (FB_3V3_OR_IO), R3.2
- new net GND: C1.2, C10.2, C11.2, C12.2, C13.2, C14.2, C15.2, C16.2, C17.2, C18.2, C19.2, C2.2, C20.2, C21.2, C22.2, C23.2, C24.2, C25.2, C26.2, C27.2, C3.2, C6.2, C7.2, C8.2, C9.2, JBT1.2 (GND), JDBG1.3 (GND), JDBG1.5 (GND), JFB1.1 (GND), JFB1.25 (SHIELD_A), JFB1.26 (SHIELD_B), JFB1.3 (GND), JPB1.1 (GND), JPB1.10 (GND), JPB1.2 (GND), JPB1.3 (GND), JPB1.4 (GND), JPB1.5 (GND), JPB1.6 (GND), JPB1.7 (GND), JPB1.8 (GND), JPB1.9 (GND), JPB1.MF_A_PIN1_51_END, JPB1.MF_A_PIN50_100_END, JPB1.MF_B_PIN1_51_END, JPB1.MF_B_PIN50_100_END, JSD1.10 (SHELL1), JSD1.11 (SHELL2), JSD1.12 (SHELL3), JSD1.13 (SHELL4), JSD1.6 (VSS), R1.2, R5.2, U1.10 (VSS), U1.27 (VSS), U1.49 (VSS), U1.74 (VSS), U1.99 (VSS), U10.1 (SDO), U10.6 (GNDIO), U10.7 (GND), U11.3 (GND), U12.2 (GND), U13.2 (GND), U2.2 (VSS), U3.12 (GND), U3.2 (A1), U3.21 (A0), U4.2 (GND), U4.9 (EP), U5.2 (SLP_N), U5.5 (GND), U6.5 (GND), U7.21 (GND), U7.24 (GND), U7.5 (GND), U8.1 (A0), U8.2 (A1), U8.3 (A2), U8.4 (VSS), U8.7 (WP), U9.5 (GND), Y1.2 (GND1), Y1.4 (GND2)
- new net IIN_SENSE: JPB1.52 (IIN_SENSE), U1.32 (PA7)
- new net IMU_INT1: U10.4 (INT1), U3.18 (P15)
- new net IOX_INT_N: R8.2, U1.54 (PB15), U3.1 (INT_N)
- new net LB_3V3_ANALOG: C4.1, C5.1, FB1.2, U1.22 (VDDA)
- new net LB_3V3_IO: JPB1.17 (LB_3V3_IO), JPB1.18 (LB_3V3_IO), R2.2, R6.1, R7.1
- new net LB_3V3_MAIN: C15.1, C16.1, C17.1, C18.1, C19.1, C2.1, C20.1, C21.1, C3.1, FB1.1, JDBG1.1 (VTREF), R2.1, R3.1, R4.1, R8.1, R9.1, U1.100 (VDD), U1.11 (VDD), U1.28 (VDD), U1.50 (VDD), U1.6 (VBAT), U1.73 (VDDUSB), U1.75 (VDD), U12.1 (VIN), U13.1 (VIN), U2.5 (VOUT), U3.24 (VCC), U4.5 (VIO), U4.8 (S), U5.3 (WAKE_N), U6.8 (VCC), U8.8 (VDD), U9.2 (VCC)
- new net LIN_RX: JPB1.74 (LIN_RX), U1.87 (PD6), U5.1 (RXD)
- new net LIN_TX: JPB1.73 (LIN_TX), U1.86 (PD5), U5.4 (TXD)
- new net MCU_HSE_IN: C9.1, U1.12 (PH0-OSC_IN), Y1.1 (XIN)
- new net MCU_HSE_OUT: C10.1, U1.13 (PH1-OSC_OUT), Y1.3 (XOUT)
- new net MCU_LSE_IN: C11.1, U1.8 (PC14-OSC32_IN), Y2.1 (XIN)
- new net MCU_LSE_OUT: C12.1, U1.9 (PC15-OSC32_OUT), Y2.2 (XOUT)
- new net MICROSD_3V3: C26.1, C27.1, JSD1.4 (VDD), R10.1, R11.1, R12.1, U12.5 (QOD), U12.6 (VOUT)
- new net MICROSD_3V3_CT: C13.1, U12.4 (CT)
- new net MICROSD_CARD_DETECT: JSD1.9 (CARD_DETECT), U3.17 (P14)
- new net MICROSD_CS_N: JSD1.2 (CD_DAT3), R12.2, U1.80 (PC12)
- new net MICROSD_DAT1: JSD1.8 (DAT1), R10.2
- new net MICROSD_DAT2: JSD1.1 (DAT2), R11.2
- new net MICROSD_PWR_EN: U1.81 (PD0), U12.3 (ON)
- new net NRST: C8.1, R15.1, R4.2, U1.14 (NRST), U3.3 (RESET_N), U9.4 (RST_N)
- new net OLED_RST_OR_INT_DNP: JFB1.24 (OLED_RST_OR_INT_DNP), U3.20 (P17)
- new net OLED_SCL: JFB1.22 (OLED_SCL), R13.2
- new net OLED_SDA: JFB1.23 (OLED_SDA), R14.2
- new net OUT10_CTL: JPB1.30 (OUT10_CTL), U1.62 (PD15)
- new net OUT10_FLT: JPB1.40 (OUT10_FLT), U1.66 (PC9)
- new net OUT10_IMON: JPB1.50 (OUT10_IMON), U1.30 (PA5)
- new net OUT1_CTL: JPB1.21 (OUT1_CTL), U1.4 (PE5)
- new net OUT1_FLT: JPB1.31 (OUT1_FLT), U1.1 (PE2)
- new net OUT1_IMON: JPB1.41 (OUT1_IMON), U1.15 (PC0)
- new net OUT2_CTL: JPB1.22 (OUT2_CTL), U1.5 (PE6)
- new net OUT2_FLT: JPB1.32 (OUT2_FLT), U1.2 (PE3)
- new net OUT2_IMON: JPB1.42 (OUT2_IMON), U1.16 (PC1)
- new net OUT3_CTL: JPB1.23 (OUT3_CTL), U1.40 (PE9)
- new net OUT3_FLT: JPB1.33 (OUT3_FLT), U1.3 (PE4)
- new net OUT3_IMON: JPB1.43 (OUT3_IMON), U1.17 (PC2)
- new net OUT4_CTL: JPB1.24 (OUT4_CTL), U1.42 (PE11)
- new net OUT4_FLT: JPB1.34 (OUT4_FLT), U1.38 (PE7)
- new net OUT4_IMON: JPB1.44 (OUT4_IMON), U1.18 (PC3)
- new net OUT5_CTL: JPB1.25 (OUT5_CTL), U1.44 (PE13)
- new net OUT5_FLT: JPB1.35 (OUT5_FLT), U1.39 (PE8)
- new net OUT5_IMON: JPB1.45 (OUT5_IMON), U1.23 (PA0)
- new net OUT6_CTL: JPB1.26 (OUT6_CTL), U1.45 (PE14)
- new net OUT6_FLT: JPB1.36 (OUT6_FLT), U1.41 (PE10)
- new net OUT6_IMON: JPB1.46 (OUT6_IMON), U1.24 (PA1)
- new net OUT7_CTL: JPB1.27 (OUT7_CTL), U1.59 (PD12)
- new net OUT7_FLT: JPB1.37 (OUT7_FLT), U1.43 (PE12)
- new net OUT7_IMON: JPB1.47 (OUT7_IMON), U1.25 (PA2)
- new net OUT8_CTL: JPB1.28 (OUT8_CTL), U1.60 (PD13)
- new net OUT8_FLT: JPB1.38 (OUT8_FLT), U1.46 (PE15)
- new net OUT8_IMON: JPB1.48 (OUT8_IMON), U1.26 (PA3)
- new net OUT9_CTL: JPB1.29 (OUT9_CTL), U1.61 (PD14)
- new net OUT9_FLT: JPB1.39 (OUT9_FLT), U1.63 (PC6)
- new net OUT9_IMON: JPB1.49 (OUT9_IMON), U1.29 (PA4)
- new net PB_5V_OUT: C1.1, JPB1.13 (PB_5V_OUT), JPB1.14 (PB_5V_OUT), JPB1.15 (PB_5V_OUT), JPB1.16 (PB_5V_OUT), U2.1 (VIN), U4.3 (VCC)
- new net PB_FAULT: JPB1.56 (PB_FAULT), U1.84 (PD3)
- new net PB_I2C_INT: JPB1.59 (PB_I2C_INT), U1.47 (PB10)
- new net PB_I2C_SCL: JPB1.57 (PB_I2C_SCL), R13.1, R6.2, U1.92 (PB6), U10.13 (SCL), U11.1 (SCL), U3.22 (SCL), U8.6 (SCL), U9.8 (SCL)
- new net PB_I2C_SDA: JPB1.58 (PB_I2C_SDA), R14.1, R7.2, U1.93 (PB7), U10.14 (SDA), U11.4 (SDA), U3.23 (SDA), U8.5 (SDA), U9.7 (SDA)
- new net PB_ID_ADC: JPB1.60 (PB_ID_ADC), U1.36 (PB1)
- new net PB_PWR_GOOD: JPB1.19 (PB_PWR_GOOD), R1.1, U1.83 (PD2), U2.3 (CE)
- new net PB_SPI_CS0: JPB1.64 (PB_SPI_CS0), U1.77 (PA15)
- new net PB_SPI_CS1: JPB1.65 (PB_SPI_CS1), U1.37 (PB2)
- new net PB_SPI_MISO: JPB1.62 (PB_SPI_MISO), JSD1.7 (DAT0), U1.90 (PB4)
- new net PB_SPI_MOSI: JPB1.63 (PB_SPI_MOSI), JSD1.3 (CMD), U1.91 (PB5)
- new net PB_SPI_SCK: JDBG1.6 (SWO), JPB1.61 (PB_SPI_SCK), JSD1.5 (CLK), U1.89 (PB3-SWO)
- new net PB_WAKE_REQ: JPB1.20 (PB_WAKE_REQ), U1.7 (PC13)
- new net RADIO_SENSOR_3V3: C22.1, C23.1, C24.1, C25.1, U10.12 (CSB), U10.5 (VDDIO), U10.8 (VDD), U11.2 (VDD), U13.5 (QOD), U13.6 (VOUT), U7.19 (VCC)
- new net RADIO_SENSOR_3V3_CT: C14.1, U13.4 (CT)
- new net RADIO_SENSOR_EN: U1.82 (PD1), U13.3 (ON)
- new net RESET_BTN: JFB1.21 (RESET_BTN), R15.2
- new net RS485_DE: JPB1.75 (RS485_DE), U1.53 (PB14), U6.2 (RE_N), U6.3 (DE)
- new net RS485_RX: JPB1.76 (RS485_RX), U1.56 (PD9), U6.1 (RO)
- new net RS485_TX: JPB1.77 (RS485_TX), U1.55 (PD8), U6.4 (DI)
- new net RTC_INT_N: U3.19 (P16), U9.3 (INT_SQW_N)
- new net SERVICE_BTN: JFB1.20 (SERVICE_BTN), U3.16 (P13)
- new net STATUS_RGB_DATA: JFB1.9 (STATUS_RGB_DATA), U3.15 (P12)
- new net SWCLK: JDBG1.4 (SWCLK), U1.76 (PA14-SWCLK)
- new net SWDIO: JDBG1.2 (SWDIO), U1.72 (PA13-SWDIO)
- new net TEMP_PCB: JPB1.53 (TEMP_PCB), U1.33 (PC4)
- new net TEMP_PWR_A: JPB1.54 (TEMP_PWR_A), U1.34 (PC5)
- new net TEMP_PWR_B: JPB1.55 (TEMP_PWR_B), U1.35 (PB0)
- new net UART_RX: JPB1.79 (UART_RX), U1.79 (PC11), U7.20 (P0.12)
- new net UART_TX: JPB1.78 (UART_TX), U1.78 (PC10), U7.22 (P0.07)
- new net USB_CC1: JFB1.6 (USB_CC1)
- new net USB_CC2: JFB1.7 (USB_CC2)
- new net USB_D_N: JFB1.5 (USB_D_N), U1.70 (PA11-USB_DM)
- new net USB_D_P: JFB1.4 (USB_D_P), U1.71 (PA12-USB_DP)
- new net USB_VBUS_SENSE: JFB1.8 (USB_VBUS_SENSE), U1.57 (PD10)
- new net VBAT_SENSE: JPB1.51 (VBAT_SENSE), U1.31 (PA6)
- new net VCAP1: C6.1, U1.48 (VCAP1)
- new net VCAP2: C7.1, U1.98 (VCAP2)
- no-connect marks 0 -> 67
Other:
- note added: "LB-100 reviewed value-bearing Rev.1 capture. STM32H563VIT6 LQFP100; exact ST package positions; JPB1 100 signals plus four GND MF circuits; PB_5V_OUT 500 mA allocation with reviewed 229.2 mA sustained and 381.2 mA service-peak budgets including FB-100 worst-case indication; ADR-0015 CAN1 FDCAN/read-only ownership with no LB transceiver; CAN1_TX_ROUTE remains the PB DNP/open route. TCA9539-Q1 maps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"
- note removed: "Blocked in this scaffold: - KiCad board import while footprint binding is open - KiCad board import while mechanical envelope is open - Gerber generation - drill files - pick-place files - BOM/CPL order package - vehicle-CAN TX enable path"
- note removed: "LB-100 schematic scaffold only. Do not create LB-100.kicad_pcb from this project until ../LB-100-pcb-layout-start-checklist.csv closes footprint binding and mechanical envelope gates. Primary inputs: - ../LB-100-requirements.md - ../LB-100-power-budget-precheck.md - ../LB-100-schematic-freeze-checklist.md - ../LB-100-pcb-layout-start-checklist.csv - ../LB-100-footprint-binding-inventory.csv - ../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"
- note removed: "Reviewed LB-100 value-bearing schematic inputs: - MCU baseline STM32H563VITx LQFP100; STM32H573VITx security alternate; STM32H563RGT6 fallback only after resource reduction. - PB_5V_OUT budget: 500 mA sustained allocation; 219.2 mA sustained LB load; 415.2 mA service peak; USB no-back-power boundary. - JPB1: exact OUT1_CTL..OUT10_CTL, OUT1_FLT..OUT10_FLT, OUT1_IMON..OUT10_IMON, PB_I2C, CAN1, CAN2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"
- note removed: "Schematic freeze evidence: - ../LB-100-schematic-review-closeout.md - ../LB-100-stm32h563-pin-binding-precheck.csv - ../LB-100-rail-budget-closeout-precheck.csv - ../LB-100-communication-safety-precheck.csv - ../LB-100-service-storage-sensor-precheck.csv - ../LB-100-mcu-sourcing-precheck.csv - ../LB-100-component-sourcing-precheck.csv - ../LB-100-pcb-layout-start-checklist.csv - ../LB-100-footpri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"
- title: LB-100 Logic Board -> LB-100 Logic Board — Value-Bearing Rev.1

Commit message: fix: reopen load dump and correct LB FB electricals
Parts:
- added C28: 1uF 6.3V X7R, LB100:R_C_0603_1608Metric, symbol LB100:LB100_C28
- added C29: 100nF 6.3V X7R, LB100:R_C_0603_1608Metric, symbol LB100:LB100_C29
- added C30: 100nF 6.3V X7R, LB100:R_C_0603_1608Metric, symbol LB100:LB100_C30
- added C31: 100nF 6.3V X7R BMI270 VDDIO, LB100:R_C_0603_1608Metric, symbol LB100:LB100_C31
- added R16: 0R, LB100:R_C_0603_1608Metric, symbol LB100:LB100_R16
- added R17: 0R single-point analog return, LB100:R_C_0603_1608Metric, symbol LB100:LB100_R17
- added U14: SN74LVC1G17QDBVRQ1, LB100:SOT-25_L3.0-W1.6-P0.95-LS2.8-TL, symbol LB100:LB100_U14
Connections:
- net ADC_REF: now also C28.1, C29.1, R16.2
- net AGND: now also C28.2, C29.2, R17.1
- net GND: now also C30.2, C31.2, R17.2, U14.3 (GND)
- net LB_3V3_ANALOG: now also R16.1
- net LB_3V3_IO: now also U10.12 (CSB), U10.5 (VDDIO), U11.2 (VDD), C30.1, C31.1, U14.5 (VCC)
- net RADIO_SENSOR_3V3: no longer U10.12 (CSB), U10.5 (VDDIO), U11.2 (VDD)
- net STATUS_RGB_DATA: now also U1.88 (PD7); no longer U3.15 (P12)
- net USB_VBUS_SENSE renamed USB_VBUS_DETECT_RAW
- net USB_VBUS_DETECT_RAW: now also U14.2 (A); no longer U1.57 (PD10)
- new net USB_VBUS_PRESENT: U1.57 (PD10), U14.4 (Y)
- no-connect marks 67 -> 68
Other:
- moved on the sheet: C1, C10, C11, C12, C13, C14, C15, C16, C17, C18, C19, C2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

Commit message: fix: isolate BLE domain and define USB detect
Parts:
- added C32: 100nF 6.3V X7R U15, LB100:R_C_0603_1608Metric, symbol LB100:LB100_C32
- added C33: 100nF 6.3V X7R U16, LB100:R_C_0603_1608Metric, symbol LB100:LB100_C33
- added C34: 100nF 6.3V X7R U17, LB100:R_C_0603_1608Metric, symbol LB100:LB100_C34
- added R18: 22k 1% switched UART idle clamp, LB100:R_C_0603_1608Metric, symbol LB100:LB100_R18
- added R19: 22k 1% switched UART idle clamp, LB100:R_C_0603_1608Metric, symbol LB100:LB100_R19
- added R20: 100k 1% MCU UART idle pull-up, LB100:R_C_0603_1608Metric, symbol LB100:LB100_R20
- added R21: 100k 1% reset default assert, LB100:R_C_0603_1608Metric, symbol LB100:LB100_R21
- added R22: 100k 1% MCU UART idle pull-up, LB100:R_C_0603_1608Metric, symbol LB100:LB100_R22
- added U15: SN74LVC1G125QDBVRQ1, LB100:SOT-25_L3.0-W1.6-P0.95-LS2.8-TL, symbol LB100:LB100_U15
- added U16: SN74LVC1G125QDBVRQ1, LB100:SOT-25_L3.0-W1.6-P0.95-LS2.8-TL, symbol LB100:LB100_U16
- added U17: SN74LVC1G125QDBVRQ1, LB100:SOT-25_L3.0-W1.6-P0.95-LS2.8-TL, symbol LB100:LB100_U17
- R9: value 10k 1% -> 10k 1% switched reset pull-up
Connections:
- net BLE_RESET_N: now also U17.4 (Y); no longer U1.97 (PE0)
- net GND: now also C32.2, C33.2, C34.2, R21.2, U15.1 (OE_N), U15.3 (GND), U16.1 (OE_N), U16.3 (GND), U17.1 (OE_N), U17.3 (GND)
- net LB_3V3_MAIN: now also R20.1, R22.1; no longer R9.1
- net RADIO_SENSOR_3V3: now also R9.1, C32.1, C33.1, C34.1, R18.2, R19.2, U15.5 (VCC), U16.5 (VCC), U17.5 (VCC)
- net UART_RX: now also R20.2, U16.4 (Y); no longer U7.20 (P0.12)
- net UART_TX: now also R22.2, U15.2 (A); no longer U7.22 (P0.07)
- new net BLE_RESET_N_MCU: R21.1, U1.97 (PE0), U17.2 (A)
- new net BLE_UART_RX_MODULE: R18.1, U15.4 (Y), U7.22 (P0.07)
- new net BLE_UART_TX_MODULE: R19.1, U16.2 (A), U7.20 (P0.12)
Other:
- moved on the sheet: C1, C10, C11, C12, C13, C14, C15, C16, C17, C18, C19, C2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

Commit message: feat(platform): authorize unified EVT development
Parts:
- added C35: 10nF 50V X7R fog input filter, LB100:R_C_0603_1608Metric, symbol LB100:LB100_C35
- added R23: 10k 1% fog input pull-up, LB100:R_C_0603_1608Metric, symbol LB100:LB100_R23
Connections:
- net GND: now also C35.2
- net LB_3V3_IO: now also R23.1
- net EXT_DIG1 renamed FOG_SW_IN
- net FOG_SW_IN: now also C35.1, R23.2
Other:
- moved on the sheet: C15, C16, C17, C18, C19, C20, C21, C22, C23, C24, C25, C26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

Commit message: feat: add dual protected fog switch inputs
Parts:
- added C36: 47nF 50V X7R FOG_B filter, LB100:R_C_0603_1608Metric, symbol LB100:LB100_C36
- added C37: 100nF 6.3V X7R U18, LB100:R_C_0603_1608Metric, symbol LB100:LB100_C37
- added C38: 100nF 6.3V X7R U19, LB100:R_C_0603_1608Metric, symbol LB100:LB100_C38
- added D18: ESD2CANFD24DBZRQ1, LB100:SOT-23-3_DBZ_TI, symbol LB100:LB100_D18
- added D19: BZT52H-B4V3-Q, LB100:SOD-123F_L2.6-W1.6, symbol LB100:LB100_D19
- added D20: BZT52H-B4V3-Q, LB100:SOD-123F_L2.6-W1.6, symbol LB100:LB100_D20
- added Q18: BC847BQ-7-F 12V OPTION, LB100:SOT-23-3_DBZ_TI, symbol LB100:LB100_Q18
- added Q19: BC847BQ-7-F 12V OPTION, LB100:SOT-23-3_DBZ_TI, symbol LB100:LB100_Q19
- added R24: 47k 1% FOG_A 12V base DNP, LB100:R_C_0603_1608Metric, symbol LB100:LB100_R24
- added R25: 100k 1% FOG_A base pull-down DNP, LB100:R_C_0603_1608Metric, symbol LB100:LB100_R25
- added R26: 47k 1% FOG_A pull-up, LB100:R_C_0603_1608Metric, symbol LB100:LB100_R26
- added R27: 4.7k 1% FOG_B dry-contact series, LB100:R_C_0603_1608Metric, symbol LB100:LB100_R27
- added R28: 47k 1% FOG_B 12V base DNP, LB100:R_C_0603_1608Metric, symbol LB100:LB100_R28
- added R29: 100k 1% FOG_B base pull-down DNP, LB100:R_C_0603_1608Metric, symbol LB100:LB100_R29
- added R30: 47k 1% FOG_B pull-up, LB100:R_C_0603_1608Metric, symbol LB100:LB100_R30
- added U18: SN74LVC1G17QDBVRQ1, LB100:SOT-25_L3.0-W1.6-P0.95-LS2.8-TL, symbol LB100:LB100_U18
- added U19: SN74LVC1G17QDBVRQ1, LB100:SOT-25_L3.0-W1.6-P0.95-LS2.8-TL, symbol LB100:LB100_U19
- C35: value 10nF 50V X7R fog input filter -> 47nF 50V X7R FOG_A filter
- R23: value 10k 1% fog input pull-up -> 4.7k 1% FOG_A dry-contact series
Connections:
- net GND: now also C36.2, C37.2, C38.2, D18.3 (GND), D19.2 (A), D20.2 (A), Q18.2 (E), Q19.2 (E), R25.2, R29.2, U18.3 (GND), U19.3 (GND)
- net LB_3V3_IO: now also C37.1, C38.1, R26.1, R30.1, U18.5 (VCC), U19.5 (VCC); no longer R23.1
- net EXT_DIG2 renamed FOG_B_SW_IN
- net FOG_B_SW_IN: now also D18.2 (IO2), R27.1, R28.1; no longer U1.68 (PA9)
- net FOG_SW_IN renamed FOG_A_FILTERED
- net FOG_A_FILTERED: now also D19.1 (K), Q18.3 (C), R26.2, U18.2 (A); no longer JPB1.82 (FOG_SW_IN), U1.67 (PA8)
- new net FOG_A_12V_BASE: Q18.1 (B), R24.2, R25.1
- new net FOG_A_SW_IN: D18.1 (IO1), JPB1.82 (FOG_A_SW_IN), R23.1, R24.1
- new net FOG_A_SW_IN_MCU: U1.67 (PA8), U18.4 (Y)
- new net FOG_B_12V_BASE: Q19.1 (B), R28.2, R29.1
- new net FOG_B_FILTERED: C36.1, D20.1 (K), Q19.3 (C), R27.2, R30.2, U19.2 (A)
- new net FOG_B_SW_IN_MCU: U1.68 (PA9), U19.4 (Y)
- no-connect marks 68 -> 70
Other:
- moved on the sheet: C1, C10, C11, C12, C13, C14, C15, C16, C17, C18, C19, C2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

Commit message: hardware: correct fog entry and EVT layout gates
Parts:
- removed D18: ESD2CANFD24DBZRQ1, LB100:SOT-23-3_DBZ_TI, symbol LB100:LB100_D18
Other:
- moved on the sheet: C1, C10, C11, C12, C13, C14, C15, C16, C17, C18, C19, C2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

Commit message: feat: add E73 recovery and persistent CAN logging
Parts:
- added TP1: E73_SWDIO, LB100:TestPoint_SMD_1.2mm, symbol LB100:LB100_TP1
- added TP2: E73_SWDCLK, LB100:TestPoint_SMD_1.2mm, symbol LB100:LB100_TP2
- added TP3: BLE_RESET_N, LB100:TestPoint_SMD_1.2mm, symbol LB100:LB100_TP3
- added TP4: RADIO_SENSOR_3V3, LB100:TestPoint_SMD_1.2mm, symbol LB100:LB100_TP4
- added TP5: GND, LB100:TestPoint_SMD_1.2mm, symbol LB100:LB100_TP5
Connections:
- net BLE_RESET_N: now also TP3.1 (BLE_RESET_N)
- net GND: now also TP5.1 (GND)
- net RADIO_SENSOR_3V3: now also TP4.1 (RADIO_SENSOR_3V3)
- net E73_SWDIO: now reaches U7.37 (SWDIO)
- net E73_SWDIO: now also TP1.1 (E73_SWDIO)
- net E73_SWDCLK: now reaches U7.39 (SWDCLK)
- net E73_SWDCLK: now also TP2.1 (E73_SWDCLK)
- no-connect marks 70 -> 68
Other:
- moved on the sheet: C1, C10, C11, C12, C13, C14, C15, C16, C17, C18, C19, C2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
