File: hardware/front-board/FB-100/kicad/FB-100.kicad_sch (KiCad schematic)
At the start: 0 parts

Commit message: Close FB USB no back power layout model
Other:
- note added: "Blocked in this scaffold: - KiCad board import while footprint binding is open - KiCad board import until layout-start checklist permits board import - Gerber generation - drill files - pick-place files - BOM/CPL order package - accessory role names in UI hardware"
- note added: "FB-100 schematic scaffold only. Do not create FB-100.kicad_pcb from this project until ../FB-100-pcb-layout-start-checklist.csv closes footprint binding. The mechanical envelope and USB/no-back-power layout inputs are closed. Primary inputs: - ../FB-100-requirements.md - ../FB-100-schematic-freeze-checklist.md - ../FB-100-pcb-layout-start-checklist.csv - ../FB-100-footprint-binding-inventory.csv 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"
- note added: "Reviewed FB-100 value-bearing schematic inputs: - JFB1 24-pin interface with USB_D_P, USB_D_N, USB_CC1, USB_CC2, USB_VBUS_SENSE, FB_3V3_IO, GND, status RGB, CH_LED_1..CH_LED_10, SERVICE_BTN, RESET_BTN, OLED_SCL, OLED_SDA. - USB-C service is device-only; CC Rd behavior; ESD protection; VBUS sense-only; no back-power into LB-100 or PB-100. - USB/no-back-power layout model is closed; ESD placement, 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"
- note added: "Schematic freeze evidence: - ../FB-100-schematic-review-closeout.md - ../FB-100-interface-signal-plan.csv - ../FB-100-interface-pinout-closeout.csv - ../FB-100-usb-service-closeout-precheck.csv - ../FB-100-ui-control-closeout-precheck.csv - ../FB-100-ui-mechanical-precheck.csv - ../FB-100-mechanical-envelope-precheck.csv - ../FB-100-mechanical-layout-inputs.csv - ../FB-100-usb-no-back-power-layou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"
- note removed: "Blocked in this scaffold: - KiCad board import while footprint binding is open - KiCad board import while mechanical envelope is open - Gerber generation - drill files - pick-place files - BOM/CPL order package - accessory role names in UI hardware"
- note removed: "FB-100 schematic scaffold only. Do not create FB-100.kicad_pcb from this project until ../FB-100-pcb-layout-start-checklist.csv closes footprint binding and mechanical envelope gates. Primary inputs: - ../FB-100-requirements.md - ../FB-100-schematic-freeze-checklist.md - ../FB-100-pcb-layout-start-checklist.csv - ../FB-100-footprint-binding-inventory.csv - ../FB-100-mechanical-envelope-inventory.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"
- note removed: "Reviewed FB-100 value-bearing schematic inputs: - JFB1 24-pin interface with USB_D_P, USB_D_N, USB_CC1, USB_CC2, USB_VBUS_SENSE, FB_3V3_IO, GND, status RGB, CH_LED_1..CH_LED_10, SERVICE_BTN, RESET_BTN, OLED_SCL, OLED_SDA. - USB-C service is device-only; CC Rd behavior; ESD protection; VBUS sense-only; no back-power into LB-100 or PB-100. - UI hardware stays role-free: channel/status indicators on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"
- note removed: "Schematic freeze evidence: - ../FB-100-schematic-review-closeout.md - ../FB-100-interface-signal-plan.csv - ../FB-100-interface-pinout-closeout.csv - ../FB-100-usb-service-closeout-precheck.csv - ../FB-100-ui-control-closeout-precheck.csv - ../FB-100-ui-mechanical-precheck.csv - ../FB-100-mechanical-envelope-precheck.csv - ../FB-100-component-sourcing-precheck.csv - ../FB-100-pcb-layout-start-che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"
Changed lines of the file:
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@@
     (comment 4 "USB service path must not back-power LB-100 or PB-100 unless reviewed.")
   )
-  (text "FB-100 schematic scaffold only.\n\nDo not create FB-100.kicad_pcb from this project until ../FB-100-pcb-layout-start-checklist.csv closes footprint binding and mechanical envelope gates.\n\nPrimary inputs:\n- ../FB-100-requirements.md\n- ../FB-100-schematic-freeze-checklist.md\n- ../FB-100-pcb-layout-start-checklist.csv\n- ../FB-100-footprint-binding-inventory.csv\n- ../FB-100-mechanical-envelope-inventory.csv\n- ../FB-100-board-release-blocker-register.csv\n- ../../../logic-board/LB-100/LB-100-requirements.md"
+  (text "FB-100 schematic scaffold only.\n\nDo not create FB-100.kicad_pcb from this project until ../FB-100-pcb-layout-start-checklist.csv closes footprint binding. The mechanical envelope and USB/no-back-power layout inputs are closed.\n\nPrimary inputs:\n- ../FB-100-requirements.md\n- ../FB-100-schematic-freeze-checklist.md\n- ../FB-100-pcb-layout-start-checklist.csv\n- ../FB-100-footprint-binding-inventory.csv\n- ../FB-100-mechanical-envelope-inventory.csv\n- ../FB-100-board-release-blocker-register.csv\n- ../../../logic-board/LB-100/LB-100-requirements.md"
     (at 25 30 0)
     (effects
@@
     )
   )
-  (text "Blocked in this scaffold:\n- KiCad board import while footprint binding is open\n- KiCad board import while mechanical envelope is open\n- Gerber generation\n- drill files\n- pick-place files\n- BOM/CPL order package\n- accessory role names in UI hardware"
+  (text "Blocked in this scaffold:\n- KiCad board import while footprint binding is open\n- KiCad board import until layout-start checklist permits board import\n- Gerber generation\n- drill files\n- pick-place files\n- BOM/CPL order package\n- accessory role names in UI hardware"
     (at 25 95 0)
     (effects
@@
     )
   )
-  (text "Reviewed FB-100 value-bearing schematic inputs:\n- JFB1 24-pin interface with USB_D_P, USB_D_N, USB_CC1, USB_CC2, USB_VBUS_SENSE, FB_3V3_IO, GND, status RGB, CH_LED_1..CH_LED_10, SERVICE_BTN, RESET_BTN, OLED_SCL, OLED_SDA.\n- USB-C service is device-only; CC Rd behavior; ESD protection; VBUS sense-only; no back-power into LB-100 or PB-100.\n- UI hardware stays role-free: channel/status indicators only, no accessory names.\n- Optional OLED remains DNP until mechanical and power review.\n- Mechanical envelope, USB access, LED/button alignment, service sealing, and enclosure boundary are reviewed."
+  (text "Reviewed FB-100 value-bearing schematic inputs:\n- JFB1 24-pin interface with USB_D_P, USB_D_N, USB_CC1, USB_CC2, USB_VBUS_SENSE, FB_3V3_IO, GND, status RGB, CH_LED_1..CH_LED_10, SERVICE_BTN, RESET_BTN, OLED_SCL, OLED_SDA.\n- USB-C service is device-only; CC Rd behavior; ESD protection; VBUS sense-only; no back-power into LB-100 or PB-100.\n- USB/no-back-power layout model is closed; ESD placement, D+/D- routing, CC behavior, VBUS sense-only routing, shield return, and JFB1 FFC transition are layout inputs.\n- UI hardware stays role-free: channel/status indicators only, no accessory names.\n- Optional OLED remains DNP unless populated by reviewed variant.\n- Mechanical envelope, USB access, LED/button alignment, service sealing, and enclosure boundary are reviewed."
     (at 130 30 0)
     (effects
@@
     )
   )
-  (text "Schematic freeze evidence:\n- ../FB-100-schematic-review-closeout.md\n- ../FB-100-interface-signal-plan.csv\n- ../FB-100-interface-pinout-closeout.csv\n- ../FB-100-usb-service-closeout-precheck.csv\n- ../FB-100-ui-control-closeout-precheck.csv\n- ../FB-100-ui-mechanical-precheck.csv\n- ../FB-100-mechanical-envelope-precheck.csv\n- ../FB-100-component-sourcing-precheck.csv\n- ../FB-100-pcb-layout-start-checklist.csv\n- ../FB-100-footprint-binding-inventory.csv\n- ../FB-100-mechanical-envelope-inventory.csv\n\nPCB layout and manufacturing outputs remain separate post-freeze work."
+  (text "Schematic freeze evidence:\n- ../FB-100-schematic-review-closeout.md\n- ../FB-100-interface-signal-plan.csv\n- ../FB-100-interface-pinout-closeout.csv\n- ../FB-100-usb-service-closeout-precheck.csv\n- ../FB-100-ui-control-closeout-precheck.csv\n- ../FB-100-ui-mechanical-precheck.csv\n- ../FB-100-mechanical-envelope-precheck.csv\n- ../FB-100-mechanical-layout-inputs.csv\n- ../FB-100-usb-no-back-power-layout-rules.csv\n- ../FB-100-component-sourcing-precheck.csv\n- ../FB-100-pcb-layout-start-checklist.csv\n- ../FB-100-footprint-binding-inventory.csv\n- ../FB-100-mechanical-envelope-inventory.csv\n\nPCB layout and manufacturing outputs remain separate post-freeze work."
     (at 130 120 0)
     (effects

Commit message: Close FB local footprint binding
Other:
- note added: "Blocked in this scaffold: - KiCad board import while schematic symbol promotion is open - KiCad board import until layout-start checklist permits board import - Gerber generation - drill files - pick-place files - BOM/CPL order package - accessory role names in UI hardware"
- note added: "FB-100 schematic scaffold only. Do not create FB-100.kicad_pcb from this project until ../FB-100-pcb-layout-start-checklist.csv closes schematic symbol promotion. Footprint binding, the mechanical envelope, and USB/no-back-power layout inputs are closed. Primary inputs: - ../FB-100-requirements.md - ../FB-100-schematic-freeze-checklist.md - ../FB-100-pcb-layout-start-checklist.csv - ../FB-100-foo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"
- note removed: "Blocked in this scaffold: - KiCad board import while footprint binding is open - KiCad board import until layout-start checklist permits board import - Gerber generation - drill files - pick-place files - BOM/CPL order package - accessory role names in UI hardware"
- note removed: "FB-100 schematic scaffold only. Do not create FB-100.kicad_pcb from this project until ../FB-100-pcb-layout-start-checklist.csv closes footprint binding. The mechanical envelope and USB/no-back-power layout inputs are closed. Primary inputs: - ../FB-100-requirements.md - ../FB-100-schematic-freeze-checklist.md - ../FB-100-pcb-layout-start-checklist.csv - ../FB-100-footprint-binding-inventory.csv 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"
Changed lines of the file:
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@@
     (comment 4 "USB service path must not back-power LB-100 or PB-100 unless reviewed.")
   )
-  (text "FB-100 schematic scaffold only.\n\nDo not create FB-100.kicad_pcb from this project until ../FB-100-pcb-layout-start-checklist.csv closes footprint binding. The mechanical envelope and USB/no-back-power layout inputs are closed.\n\nPrimary inputs:\n- ../FB-100-requirements.md\n- ../FB-100-schematic-freeze-checklist.md\n- ../FB-100-pcb-layout-start-checklist.csv\n- ../FB-100-footprint-binding-inventory.csv\n- ../FB-100-mechanical-envelope-inventory.csv\n- ../FB-100-board-release-blocker-register.csv\n- ../../../logic-board/LB-100/LB-100-requirements.md"
+  (text "FB-100 schematic scaffold only.\n\nDo not create FB-100.kicad_pcb from this project until ../FB-100-pcb-layout-start-checklist.csv closes schematic symbol promotion. Footprint binding, the mechanical envelope, and USB/no-back-power layout inputs are closed.\n\nPrimary inputs:\n- ../FB-100-requirements.md\n- ../FB-100-schematic-freeze-checklist.md\n- ../FB-100-pcb-layout-start-checklist.csv\n- ../FB-100-footprint-binding-inventory.csv\n- ../FB-100-footprint-binding-closeout.csv\n- ../FB-100-mechanical-envelope-inventory.csv\n- ../FB-100-board-release-blocker-register.csv\n- ../../../logic-board/LB-100/LB-100-requirements.md"
     (at 25 30 0)
     (effects
@@
     )
   )
-  (text "Blocked in this scaffold:\n- KiCad board import while footprint binding is open\n- KiCad board import until layout-start checklist permits board import\n- Gerber generation\n- drill files\n- pick-place files\n- BOM/CPL order package\n- accessory role names in UI hardware"
+  (text "Blocked in this scaffold:\n- KiCad board import while schematic symbol promotion is open\n- KiCad board import until layout-start checklist permits board import\n- Gerber generation\n- drill files\n- pick-place files\n- BOM/CPL order package\n- accessory role names in UI hardware"
     (at 25 95 0)
     (effects
@@
     )
   )
-  (text "Reviewed FB-100 value-bearing schematic inputs:\n- JFB1 24-pin interface with USB_D_P, USB_D_N, USB_CC1, USB_CC2, USB_VBUS_SENSE, FB_3V3_IO, GND, status RGB, CH_LED_1..CH_LED_10, SERVICE_BTN, RESET_BTN, OLED_SCL, OLED_SDA.\n- USB-C service is device-only; CC Rd behavior; ESD protection; VBUS sense-only; no back-power into LB-100 or PB-100.\n- USB/no-back-power layout model is closed; ESD placement, D+/D- routing, CC behavior, VBUS sense-only routing, shield return, and JFB1 FFC transition are layout inputs.\n- UI hardware stays role-free: channel/status indicators only, no accessory names.\n- Optional OLED remains DNP unless populated by reviewed variant.\n- Mechanical envelope, USB access, LED/button alignment, service sealing, and enclosure boundary are reviewed."
+  (text "Reviewed FB-100 value-bearing schematic inputs:\n- JFB1 24-pin interface with USB_D_P, USB_D_N, USB_CC1, USB_CC2, USB_VBUS_SENSE, FB_3V3_IO, GND, status RGB, CH_LED_1..CH_LED_10, SERVICE_BTN, RESET_BTN, OLED_SCL, OLED_SDA.\n- USB-C service is device-only; CC Rd behavior; ESD protection; VBUS sense-only; no back-power into LB-100 or PB-100.\n- USB/no-back-power layout model is closed; ESD placement, D+/D- routing, CC behavior, VBUS sense-only routing, shield return, and JFB1 FFC transition are layout inputs.\n- footprint binding is closed in FB100.pretty but schematic symbol promotion remains open.\n- UI hardware stays role-free: channel/status indicators only, no accessory names.\n- Optional OLED remains DNP unless populated by reviewed variant.\n- Mechanical envelope, USB access, LED/button alignment, service sealing, and enclosure boundary are reviewed."
     (at 130 30 0)
     (effects
@@
     )
   )
-  (text "Schematic freeze evidence:\n- ../FB-100-schematic-review-closeout.md\n- ../FB-100-interface-signal-plan.csv\n- ../FB-100-interface-pinout-closeout.csv\n- ../FB-100-usb-service-closeout-precheck.csv\n- ../FB-100-ui-control-closeout-precheck.csv\n- ../FB-100-ui-mechanical-precheck.csv\n- ../FB-100-mechanical-envelope-precheck.csv\n- ../FB-100-mechanical-layout-inputs.csv\n- ../FB-100-usb-no-back-power-layout-rules.csv\n- ../FB-100-component-sourcing-precheck.csv\n- ../FB-100-pcb-layout-start-checklist.csv\n- ../FB-100-footprint-binding-inventory.csv\n- ../FB-100-mechanical-envelope-inventory.csv\n\nPCB layout and manufacturing outputs remain separate post-freeze work."
+  (text "Schematic freeze evidence:\n- ../FB-100-schematic-review-closeout.md\n- ../FB-100-interface-signal-plan.csv\n- ../FB-100-interface-pinout-closeout.csv\n- ../FB-100-usb-service-closeout-precheck.csv\n- ../FB-100-ui-control-closeout-precheck.csv\n- ../FB-100-ui-mechanical-precheck.csv\n- ../FB-100-mechanical-envelope-precheck.csv\n- ../FB-100-mechanical-layout-inputs.csv\n- ../FB-100-usb-no-back-power-layout-rules.csv\n- ../FB-100-component-sourcing-precheck.csv\n- ../FB-100-pcb-layout-start-checklist.csv\n- ../FB-100-footprint-binding-inventory.csv\n- ../FB-100-footprint-binding-closeout.csv\n- ../FB-100-mechanical-envelope-inventory.csv\n\nPCB layout and manufacturing outputs remain separate post-freeze work."
     (at 130 120 0)
     (effects

Commit message: feat(hardware): close LB FB schematics and FX18 mechanics
Parts:
- added C1: 100nF 16V X7R, FB100:R_C_0603_1608Metric, symbol FB100:FB100_C1
- added C2: 1nF 1kV C0G, FB100:R_C_0603_1608Metric, symbol FB100:FB100_C2
- added C3: 1uF 6.3V X7R, FB100:R_C_0603_1608Metric, symbol FB100:FB100_C3
- added C4: 1uF 6.3V X7R, FB100:R_C_0603_1608Metric, symbol FB100:FB100_C4
- added C5: 1uF 6.3V X7R, FB100:R_C_0603_1608Metric, symbol FB100:FB100_C5
- added C6: 100nF 6.3V X7R, FB100:R_C_0603_1608Metric, symbol FB100:FB100_C6
- added C7: 100nF 6.3V X7R, FB100:R_C_0603_1608Metric, symbol FB100:FB100_C7
- added D1: USBLC6-2SC6, FB100:SOT-23-6_L2.9-W1.6-P0.95-LS2.8-BL, symbol FB100:FB100_D1
- added D10: KT-0805Y, FB100:LED0805-R-RD, symbol FB100:FB100_D10
- added D11: KT-0805Y, FB100:LED0805-R-RD, symbol FB100:FB100_D11
- added D12: KT-0805Y, FB100:LED0805-R-RD, symbol FB100:FB100_D12
- added D2: 19-237/R6GHBHC-A01/2T, FB100:LED-ARRAY-SMD_4P-L1.6-W1.6-BL_1, symbol FB100:FB100_D2
- added D3: KT-0805Y, FB100:LED0805-R-RD, symbol FB100:FB100_D3
- added D4: KT-0805Y, FB100:LED0805-R-RD, symbol FB100:FB100_D4
- added D5: KT-0805Y, FB100:LED0805-R-RD, symbol FB100:FB100_D5
- added D6: KT-0805Y, FB100:LED0805-R-RD, symbol FB100:FB100_D6
- added D7: KT-0805Y, FB100:LED0805-R-RD, symbol FB100:FB100_D7
- added D8: KT-0805Y, FB100:LED0805-R-RD, symbol FB100:FB100_D8
- added D9: KT-0805Y, FB100:LED0805-R-RD, symbol FB100:FB100_D9
- added J1: USB4105-GF-A, FB100:TYPE-C-SMD_SBC-160S1A-20-S412, symbol FB100:FB100_J1
- added J2: SSD1306_I2C_MODULE_DNP, FB100:PinHeader_1x04_P2.54mm_Vertical, symbol FB100:FB100_J2
- added JFB1: AFC07-S24ECA-00, FB100:FPC-SMD_AFC07-S24ECA-00, symbol FB100:FB100_JFB1
- added R1: 1k 1%, FB100:R_C_0603_1608Metric, symbol FB100:FB100_R1
- added R10: 1k 1%, FB100:R_C_0603_1608Metric, symbol FB100:FB100_R10
- added R11: 5.1k 1%, FB100:R_C_0603_1608Metric, symbol FB100:FB100_R11
- added R12: 5.1k 1%, FB100:R_C_0603_1608Metric, symbol FB100:FB100_R12
- added R13: 100k 1%, FB100:R_C_0603_1608Metric, symbol FB100:FB100_R13
- added R14: 27k 1%, FB100:R_C_0603_1608Metric, symbol FB100:FB100_R14
- added R15: 1M 1%, FB100:R_C_0603_1608Metric, symbol FB100:FB100_R15
- added R16: 35.7k 1%, FB100:R_C_0603_1608Metric, symbol FB100:FB100_R16
- added R17: 10k 1%, FB100:R_C_0603_1608Metric, symbol FB100:FB100_R17
- added R18: 10k 1%, FB100:R_C_0603_1608Metric, symbol FB100:FB100_R18
- added R19: 100k 1%, FB100:R_C_0603_1608Metric, symbol FB100:FB100_R19
- added R2: 1k 1%, FB100:R_C_0603_1608Metric, symbol FB100:FB100_R2
- added R3: 1k 1%, FB100:R_C_0603_1608Metric, symbol FB100:FB100_R3
- added R4: 1k 1%, FB100:R_C_0603_1608Metric, symbol FB100:FB100_R4
- added R5: 1k 1%, FB100:R_C_0603_1608Metric, symbol FB100:FB100_R5
- added R6: 1k 1%, FB100:R_C_0603_1608Metric, symbol FB100:FB100_R6
- added R7: 1k 1%, FB100:R_C_0603_1608Metric, symbol FB100:FB100_R7
- added R8: 1k 1%, FB100:R_C_0603_1608Metric, symbol FB100:FB100_R8
- added R9: 1k 1%, FB100:R_C_0603_1608Metric, symbol FB100:FB100_R9
- added SW1: EVPBB4A9B000 SERVICE, FB100:KEY-SMD_L2.6-W1.6-P0.75-LS3.0, symbol FB100:FB100_SW1
- added SW2: EVPBB4A9B000 RESET, FB100:KEY-SMD_L2.6-W1.6-P0.75-LS3.0, symbol FB100:FB100_SW2
- added U1: LTC3212EDDB#TRPBF, FB100:DFN-12-1EP_2x3mm_P0.45mm, symbol FB100:FB100_U1
Connections:
- new net CH_LED_1: D3.2 (K), JFB1.10 (CH_LED_1)
- new net CH_LED_10: D12.2 (K), JFB1.19 (CH_LED_10)
- new net CH_LED_10_A: D12.1 (A), R10.2
- new net CH_LED_1_A: D3.1 (A), R1.2
- new net CH_LED_2: D4.2 (K), JFB1.11 (CH_LED_2)
- new net CH_LED_2_A: D4.1 (A), R2.2
- new net CH_LED_3: D5.2 (K), JFB1.12 (CH_LED_3)
- new net CH_LED_3_A: D5.1 (A), R3.2
- new net CH_LED_4: D6.2 (K), JFB1.13 (CH_LED_4)
- new net CH_LED_4_A: D6.1 (A), R4.2
- new net CH_LED_5: D7.2 (K), JFB1.14 (CH_LED_5)
- new net CH_LED_5_A: D7.1 (A), R5.2
- new net CH_LED_6: D8.2 (K), JFB1.15 (CH_LED_6)
- new net CH_LED_6_A: D8.1 (A), R6.2
- new net CH_LED_7: D9.2 (K), JFB1.16 (CH_LED_7)
- new net CH_LED_7_A: D9.1 (A), R7.2
- new net CH_LED_8: D10.2 (K), JFB1.17 (CH_LED_8)
- new net CH_LED_8_A: D10.1 (A), R8.2
- new net CH_LED_9: D11.2 (K), JFB1.18 (CH_LED_9)
- new net CH_LED_9_A: D11.1 (A), R9.2
- new net FB_3V3_OR_IO: C3.1, J2.2 (VCC), JFB1.2 (FB_3V3_OR_IO), R1.1, R10.1, R17.1, R18.1, R2.1, R3.1, R4.1, R5.1, R6.1, R7.1, R8.1, R9.1, U1.12 (VIN), U1.4 (ISETB), U1.5 (ISETR)
- new net GND: C1.2, C2.2, C3.2, C5.2, C6.2, C7.2, D1.2 (GND), J1.A1 (GND), J1.A12 (GND), J1.B1 (GND), J1.B12 (GND), J2.1 (GND), JFB1.1 (GND), JFB1.25 (SHIELD_A), JFB1.26 (SHIELD_B), JFB1.3 (GND), R11.2, R12.2, R14.2, R15.2, R16.2, R19.2, SW1.B, SW1.B1, SW2.B, SW2.B1, U1.10 (GND), U1.13 (EP)
- new net OLED_RST_OR_INT_DNP: JFB1.24 (OLED_RST_OR_INT_DNP), R19.1
- new net OLED_SCL: J2.3 (SCL), JFB1.22 (OLED_SCL)
- new net OLED_SDA: J2.4 (SDA), JFB1.23 (OLED_SDA)
- new net RESET_BTN: C7.1, JFB1.21 (RESET_BTN), R18.2, SW2.A, SW2.A1
- new net RGB_B_K: D2.4 (BLUE_K), U1.9 (LEDB)
- new net RGB_CM: C4.2, U1.11 (CM)
- new net RGB_CP: C4.1, U1.1 (CP)
- new net RGB_G_K: D2.3 (GREEN_K), U1.7 (LEDG)
- new net RGB_ISETG: R16.1, U1.6 (ISETG)
- new net RGB_LED_ANODE: C5.1, D2.1 (COMMON_ANODE), U1.2 (CPO)
- new net RGB_R_K: D2.2 (RED_K), U1.8 (LEDR)
- new net SERVICE_BTN: C6.1, JFB1.20 (SERVICE_BTN), R17.2, SW1.A, SW1.A1
- new net STATUS_RGB_DATA: JFB1.9 (STATUS_RGB_DATA), U1.3 (LEDEN)
- new net USB_CC1: J1.A5 (CC1), JFB1.6 (USB_CC1), R11.1
- new net USB_CC2: J1.B5 (CC2), JFB1.7 (USB_CC2), R12.1
- new net USB_D_N: D1.4 (I_O2_OUT), JFB1.5 (USB_D_N)
- new net USB_D_N_CONN: D1.3 (I_O2_IN), J1.A7 (D-), J1.B7 (D-)
- new net USB_D_P: D1.6 (I_O1_OUT), JFB1.4 (USB_D_P)
- new net USB_D_P_CONN: D1.1 (I_O1_IN), J1.A6 (D+), J1.B6 (D+)
- new net USB_SHIELD: C2.1, J1.1 (SHIELD1), J1.2 (SHIELD2), J1.3 (SHIELD3), J1.4 (SHIELD4), R15.1
- new net USB_VBUS: D1.5 (VBUS), J1.A4 (VBUS), J1.A9 (VBUS), J1.B4 (VBUS), J1.B9 (VBUS), R13.1
- new net USB_VBUS_SENSE: C1.1, JFB1.8 (USB_VBUS_SENSE), R13.2, R14.1
- no-connect marks 0 -> 2
Other:
- note added: "FB-100 reviewed value-bearing Rev.1 capture. USB-C is USB2 device-only with two 5.1k Rd resistors, USBLC6-2SC6 flow-through ESD, VBUS sense-only divider, and no connection from USB VBUS to FB_3V3_OR_IO. LTC3212 converts the approved STATUS_RGB_DATA single wire into three regulated cathode currents for the common-anode RGB LED. CH_LED_1..CH_LED_10 remain role-free and default off while LB TCA9539-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"
- note removed: "Blocked in this scaffold: - KiCad board import while schematic symbol promotion is open - KiCad board import until layout-start checklist permits board import - Gerber generation - drill files - pick-place files - BOM/CPL order package - accessory role names in UI hardware"
- note removed: "FB-100 schematic scaffold only. Do not create FB-100.kicad_pcb from this project until ../FB-100-pcb-layout-start-checklist.csv closes schematic symbol promotion. Footprint binding, the mechanical envelope, and USB/no-back-power layout inputs are closed. Primary inputs: - ../FB-100-requirements.md - ../FB-100-schematic-freeze-checklist.md - ../FB-100-pcb-layout-start-checklist.csv - ../FB-100-foo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"
- note removed: "Reviewed FB-100 value-bearing schematic inputs: - JFB1 24-pin interface with USB_D_P, USB_D_N, USB_CC1, USB_CC2, USB_VBUS_SENSE, FB_3V3_IO, GND, status RGB, CH_LED_1..CH_LED_10, SERVICE_BTN, RESET_BTN, OLED_SCL, OLED_SDA. - USB-C service is device-only; CC Rd behavior; ESD protection; VBUS sense-only; no back-power into LB-100 or PB-100. - USB/no-back-power layout model is closed; ESD placement, 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"
- note removed: "Schematic freeze evidence: - ../FB-100-schematic-review-closeout.md - ../FB-100-interface-signal-plan.csv - ../FB-100-interface-pinout-closeout.csv - ../FB-100-usb-service-closeout-precheck.csv - ../FB-100-ui-control-closeout-precheck.csv - ../FB-100-ui-mechanical-precheck.csv - ../FB-100-mechanical-envelope-precheck.csv - ../FB-100-mechanical-layout-inputs.csv - ../FB-100-usb-no-back-power-layou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"
- title: FB-100 Front Panel Board -> FB-100 Front Panel — Value-Bearing Rev.1

Commit message: fix: reopen load dump and correct LB FB electricals
Parts:
- removed R14: 27k 1%, FB100:R_C_0603_1608Metric, symbol FB100:FB100_R14
- R13: value 100k 1% -> 100k 1% current limit
Connections:
- net USB_VBUS_SENSE renamed USB_VBUS_DETECT_RAW
Other:
- note added: "FB-100 reviewed value-bearing Rev.1 capture. USB-C is USB2 device-only with two 5.1k Rd resistors, USBLC6-2SC6 flow-through ESD, current-limited VBUS detect, and no connection from USB VBUS to FB_3V3_OR_IO. LTC3212 converts the approved STATUS_RGB_DATA single wire into three regulated cathode currents for the common-anode RGB LED. CH_LED_1..CH_LED_10 remain role-free and default off while LB TCA9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"
- note removed: "FB-100 reviewed value-bearing Rev.1 capture. USB-C is USB2 device-only with two 5.1k Rd resistors, USBLC6-2SC6 flow-through ESD, VBUS sense-only divider, and no connection from USB VBUS to FB_3V3_OR_IO. LTC3212 converts the approved STATUS_RGB_DATA single wire into three regulated cathode currents for the common-anode RGB LED. CH_LED_1..CH_LED_10 remain role-free and default off while LB TCA9539-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"
- moved on the sheet: C1, C2, C3, C4, C5, C6, C7, R15, R16, R17, R18, R19

Commit message: fix: isolate BLE domain and define USB detect
Parts:
- added R14: 15k 1% defined pulldown, FB100:R_C_0603_1608Metric, symbol FB100:FB100_R14
- C1: value 100nF 16V X7R -> 100nF 16V X7R 10%
- R13: value 100k 1% current limit -> 3.9k 1% current limit
Connections:
- net GND: now also R14.2
- net USB_VBUS_DETECT_RAW: now also R14.1
Other:
- moved on the sheet: C1, C2, C3, C4, C5, C6, C7, R15, R16, R17, R18, R19
