File: hardware/front-board/FB-100/kicad/FB-100.kicad_sch (KiCad schematic)
At the start: 44 parts, among them J1 USB4105-GF-A, J2 SSD1306_I2C_MODULE_DNP, SW1 EVPBB4A9B000 SERVICE, SW2 EVPBB4A9B000 RESET, U1 LTC3212EDDB#TRPBF

Commit message: feat(platform): authorize unified EVT development
Changed lines of the file:
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@@
     (comment 2 "Generated deterministically from accepted contracts and component decisions.")
   )
-  (text "FB-100 reviewed value-bearing Rev.1 capture. USB-C is USB2 device-only with two 5.1k Rd resistors, USBLC6-2SC6 flow-through ESD, current-limited VBUS detect, and no connection from USB VBUS to FB_3V3_OR_IO. LTC3212 converts the approved STATUS_RGB_DATA single wire into three regulated cathode currents for the common-anode RGB LED. CH_LED_1..CH_LED_10 remain role-free and default off while LB TCA9539-Q1 ports are inputs. OLED is an optional four-wire I2C module header and is DNP by default. JFB1 uses the approved 24-pin contract. Reviewed footprint binding and mechanical envelope remain governed by FB-100-pcb-layout-start-checklist.csv, FB-100-footprint-binding-inventory.csv, and FB-100-mechanical-envelope-inventory.csv. A controlled FB-100.kicad_pcb placement exists under LAYOUT-ONLY authorization. Do not create Gerbers, drills, pick-place, BOM/CPL order packages, or other manufacturing outputs. PCB layout and manufacturing outputs remain separate."
+  (text "FB-100 reviewed value-bearing Rev.1 capture. USB-C is USB2 device-only with two 5.1k Rd resistors, USBLC6-2SC6 flow-through ESD, current-limited VBUS detect, and no connection from USB VBUS to FB_3V3_OR_IO. LTC3212 converts the approved STATUS_RGB_DATA single wire into three regulated cathode currents for the common-anode RGB LED. CH_LED_1..CH_LED_10 remain role-free and default off while LB TCA9539-Q1 ports are inputs. OLED is an optional four-wire I2C module header and is DNP by default. JFB1 uses the approved 24-pin contract. Reviewed footprint binding and mechanical envelope remain governed by FB-100-pcb-layout-start-checklist.csv, FB-100-footprint-binding-inventory.csv, and FB-100-mechanical-envelope-inventory.csv. A controlled FB-100.kicad_pcb placement exists under EVT-LAYOUT-AUTHORIZED status. Do not create Gerbers, drills, pick-place, BOM/CPL order packages, or other manufacturing outputs. PCB layout and manufacturing outputs remain separate."
     (at 20 20 0)
     (effects (font (size 1.6 1.6)) (justify left top))
