File: hardware/power-board/PB-100/qualification/Q2-C100/kicad/Q2-C100.kicad_pcb (KiCad board)
At the start: 4 copper layers, 80 x 100 mm, 30 parts

Commit message: feat(pb100): complete Q2 coupon electrical routing
Parts:
- ROV1, ROV2: footprint Q2C100:R_C_0603_1608Metric -> Q2C100:R_1206_3216Metric
- moved CCAP 5.32 mm to (21.0, 39.5), turned to 90 degrees
- moved ROV3 4.00 mm to (57.0, 34.0)
- moved ROV2 2.00 mm to (57.0, 26.0)
Routing:
- net GND: track 0.00 -> 271.6 mm, vias 0 -> 10
- net CTRL_OV: track 0.00 -> 116.8 mm, vias 0 -> 1
- net CTRL_VS: track 0.00 -> 106.0 mm, vias 0 -> 4
- net SYSTEM_OUT: track 41.5 -> 123.5 mm, vias 4 -> 6
- net Q2_HGATE: track 20.4 -> 58.0 mm
- net RAW_101V: track 37.5 -> 71.1 mm
- net CTRL_FLT_N: track 0.00 -> 28.7 mm, vias 0 -> 1
- net OV_MID: track 0.00 -> 19.5 mm
- net COMMON_SOURCE: track 163.8 -> 174.6 mm, vias 12 -> 13
- net CTRL_CAP: track 0.00 -> 5.85 mm
Other:
- board text added: "PAD-TO-PAD ROUTING COMPLETE; FAB REVIEW OPEN"
- board text removed: "CRITICAL POWER + GATE LOOP ROUTED; FIXTURE NETS OPEN"

Commit message: feat(q2): strengthen coupon pre-fab evidence
Parts:
- CCAP: value 100nF 25V X7R AEC-Q200 -> CGA3E2X7R1H104K080AE 100nF 50V X7R
- ROV1, ROV2: value 42.2k 1% AEC-Q200 -> CRCW120642K2FKEAHP 42.2k 1%
- ROV3: value 1.00k 1% AEC-Q200 -> CRCW06031K00FKEAHP 1.00k 1%
- RVS: value 10.0k 1% 1206 AEC-Q200 -> CRCW120610K0FKEAHP 10.0k 1%
Routing:
- net COMMON_SOURCE: track 174.6 -> 217.9 mm, vias 13 -> 29
- net SYSTEM_OUT: vias 6 -> 9
- net RAW_101V: vias 4 -> 7

Commit message: feat(q2): bind coupon fixture interfaces
Parts:
- JDRIVE: value FORCED_DRIVER_KELVIN -> 436500428 MICRO-FIT 4POS DRIVER; footprint Q2C100:PinHeader_1x04_P2.54 -> Q2C100:MicroFit_43650_0428_Vertical_R90
- JHEAT: value ISOLATED_CASE_HEATER -> 436500228 MICRO-FIT 2POS HEATER; footprint Q2C100:PinHeader_1x02_P2.54 -> Q2C100:MicroFit_43650_0228_Vertical
- JTEMP: value ISOLATED_TSEP_INPUT -> 436500328 MICRO-FIT 3POS TEMP; footprint Q2C100:PinHeader_1x02_P2.54 -> Q2C100:MicroFit_43650_0328_Vertical
- TPD: value QDUT_DRAIN_KELVIN -> S1751-46R QDUT_DRAIN_KELVIN; footprint Q2C100:TestPoint_Loop_1.0mm -> Q2C100:Harwin_S1751-46R
- TPFLT: value FAULT_PROBE -> S1751-46R FAULT_PROBE; footprint Q2C100:TestPoint_Loop_1.0mm -> Q2C100:Harwin_S1751-46R
- TPG: value QDUT_GATE_KELVIN -> S1751-46R QDUT_GATE_KELVIN; footprint Q2C100:TestPoint_Loop_1.0mm -> Q2C100:Harwin_S1751-46R
- TPGND: value PROBE_GND -> S1751-46R PROBE_GND; footprint Q2C100:TestPoint_Loop_1.0mm -> Q2C100:Harwin_S1751-46R
- TPHG: value UCTRL_HGATE_PROBE -> S1751-46R UCTRL_HGATE_PROBE; footprint Q2C100:TestPoint_Loop_1.0mm -> Q2C100:Harwin_S1751-46R
- TPOUT: value SYSTEM_OUT_PROBE -> S1751-46R SYSTEM_OUT_PROBE; footprint Q2C100:TestPoint_Loop_1.0mm -> Q2C100:Harwin_S1751-46R
- TPOV: value OV_TRIGGER_PROBE -> S1751-46R OV_TRIGGER_PROBE; footprint Q2C100:TestPoint_Loop_1.0mm -> Q2C100:Harwin_S1751-46R
- TPS: value QDUT_SOURCE_KELVIN -> S1751-46R QDUT_SOURCE_KELVIN; footprint Q2C100:TestPoint_Loop_1.0mm -> Q2C100:Harwin_S1751-46R
- TPVS: value CTRL_VS_PROBE -> S1751-46R CTRL_VS_PROBE; footprint Q2C100:TestPoint_Loop_1.0mm -> Q2C100:Harwin_S1751-46R
- moved JTEMP 5.00 mm to (69.0, 87.0)
- moved JDRIVE 2.00 mm to (6.00, 48.0), turned to 0 degrees
- moved TPG 1.00 mm to (31.0, 35.0)
Routing:
- net GND: track 271.6 -> 287.6 mm, vias 10 -> 11
- net COMMON_SOURCE: track 217.9 -> 220.1 mm
- net Q2_HGATE: track 58.0 -> 60.2 mm
- net SYSTEM_OUT: vias 9 -> 10
- net CTRL_VS: vias 4 -> 5
- net CTRL_OV: vias 1 -> 2
- net CTRL_FLT_N: vias 1 -> 2
